File: int1/temp-luz/_autosave-temp-luz.sch (KiCad schematic (older format))
At the start: 6 parts

Commit message: DHT22PCB
Parts:
- added R?: 4.7k, symbol Device:R
- added R?: 1k, symbol Device:R
- C?: value C -> 0.1u
- R? (x2): value R -> 4.7k
Connections:
- net at IC?.1 (VCC), R?.1: now also R?.1, R?.1
- net at IC?.4 (SDA): now also R?.2
- net at IC?.6 (SCL): now also R?.2
Changed lines of the file:
@@
 P 8650 1850
 F 0 "R?" H 8720 1896 50  0000 L CNN
-F 1 "R" H 8720 1805 50  0000 L CNN
+F 1 "4.7k" H 8720 1805 50  0000 L CNN
 F 2 "" V 8580 1850 50  0001 C CNN
 F 3 "~" H 8650 1850 50  0001 C CNN
@@
 P 8650 2650
 F 0 "C?" H 8765 2696 50  0000 L CNN
-F 1 "C" H 8765 2605 50  0000 L CNN
+F 1 "0.1u" H 8765 2605 50  0000 L CNN
 F 2 "" H 8688 2500 50  0001 C CNN
 F 3 "~" H 8650 2650 50  0001 C CNN
@@
 P 6800 2550
 F 0 "R?" H 6870 2596 50  0000 L CNN
-F 1 "R" H 6870 2505 50  0000 L CNN
+F 1 "4.7k" H 6870 2505 50  0000 L CNN
 F 2 "" V 6730 2550 50  0001 C CNN
 F 3 "~" H 6800 2550 50  0001 C CNN
@@
 	1    0    0    -1
 $EndComp
+$Comp
+L Device:R R?
+U 1 1 619FCBEE
+P 8950 1850
+F 0 "R?" H 9020 1896 50  0000 L CNN
+F 1 "4.7k" H 9020 1805 50  0000 L CNN
+F 2 "" V 8880 1850 50  0001 C CNN
+F 3 "~" H 8950 1850 50  0001 C CNN
+	1    8950 1850
+	1    0    0    -1
+$EndComp
+$Comp
+L Device:R R?
+U 1 1 619FD513
+P 9250 1850
+F 0 "R?" H 9320 1896 50  0000 L CNN
+F 1 "1k" H 9320 1805 50  0000 L CNN
+F 2 "" V 9180 1850 50  0001 C CNN
+F 3 "~" H 9250 1850 50  0001 C CNN
+	1    9250 1850
+	1    0    0    -1
+$EndComp
+Wire Wire Line
+	8950 1700 8950 1500
+Wire Wire Line
+	8950 1500 8650 1500
+Connection ~ 8650 1500
+Wire Wire Line
+	9250 1700 9250 1500
+Wire Wire Line
+	9250 1500 8950 1500
+Connection ~ 8950 1500
+Wire Wire Line
+	8250 2250 8950 2250
+Wire Wire Line
+	8950 2250 8950 2000
+Wire Wire Line
+	8250 2450 9250 2450
+Wire Wire Line
+	9250 2450 9250 2000
 $EndSCHEMATC
