File: Diseño PCB/PCB-ESP32S/ModuloReles.sch (KiCad schematic (older format))
At the start: 8 parts

Commit message: Humedad y luz
Parts:
- gave numbers to parts that had none: 8
Changed lines of the file:
@@
 $Descr A4 11693 8268
 encoding utf-8
-Sheet 4 4
+Sheet 4 5
 Title ""
 Date ""
@@
 $EndDescr
 $Comp
-L Device:R R?
+L Device:R R6
 U 1 1 61A67A98
 P 3650 3150
-F 0 "R?" H 3720 3196 50  0000 L CNN
+F 0 "R6" H 3720 3196 50  0000 L CNN
 F 1 "R" H 3720 3105 50  0000 L CNN
 F 2 "" V 3580 3150 50  0001 C CNN
@@
 $EndComp
 $Comp
-L Diode:1N4007 D?
+L Diode:1N4007 D2
 U 1 1 61A68714
 P 4250 2450
-F 0 "D?" V 4204 2530 50  0000 L CNN
+F 0 "D2" V 4204 2530 50  0000 L CNN
 F 1 "1N4007" V 4295 2530 50  0000 L CNN
 F 2 "Diode_THT:D_DO-41_SOD81_P10.16mm_Horizontal" H 4250 2275 50  0001 C CNN
@@
 $EndComp
 $Comp
-L MMBT2222A:MMBT2222A Q?
+L MMBT2222A:MMBT2222A Q1
 U 1 1 61A825BF
 P 4150 3150
-F 0 "Q?" H 4294 3196 50  0000 L CNN
+F 0 "Q1" H 4294 3196 50  0000 L CNN
 F 1 "MMBT2222A" H 4294 3105 50  0000 L CNN
 F 2 "SOT23" H 4150 3150 50  0001 L BNN
@@
 $EndComp
 $Comp
-L Rele12V:SRD-05VDC-SL-C K?
+L Rele12V:SRD-05VDC-SL-C K1
 U 1 1 61A82FC5
 P 4900 2400
-F 0 "K?" H 4900 2767 50  0000 C CNN
+F 0 "K1" H 4900 2767 50  0000 C CNN
 F 1 "SRD-05VDC-SL-C" H 4900 2676 50  0000 C CNN
 F 2 "RELAY_SRD-05VDC-SL-C" H 4900 2400 50  0001 L BNN
@@
 $EndComp
 $Comp
-L Isolator:PC817 U?
+L Isolator:PC817 U3
 U 1 1 61A84C62
 P 2900 3050
-F 0 "U?" H 2900 3375 50  0000 C CNN
+F 0 "U3" H 2900 3375 50  0000 C CNN
 F 1 "PC817" H 2900 3284 50  0000 C CNN
 F 2 "Package_DIP:DIP-4_W7.62mm" H 2700 2850 50  0001 L CIN
@@
 $EndComp
 $Comp
-L Device:LED D?
+L Device:LED D1
 U 1 1 61A85954
 P 2000 3150
-F 0 "D?" H 1993 3367 50  0000 C CNN
+F 0 "D1" H 1993 3367 50  0000 C CNN
 F 1 "LED" H 1993 3276 50  0000 C CNN
 F 2 "" H 2000 3150 50  0001 C CNN
@@
 $EndComp
 $Comp
-L Device:R R?
+L Device:R R5
 U 1 1 61A8CFB4
 P 2300 2350
-F 0 "R?" H 2370 2396 50  0000 L CNN
+F 0 "R5" H 2370 2396 50  0000 L CNN
 F 1 "R" H 2370 2305 50  0000 L CNN
 F 2 "" V 2230 2350 50  0001 C CNN
@@
 $EndComp
 $Comp
-L Connector:Screw_Terminal_01x03 J?
+L Connector:Screw_Terminal_01x03 J1
 U 1 1 61A8F333
 P 5900 2300
-F 0 "J?" H 5980 2342 50  0000 L CNN
+F 0 "J1" H 5980 2342 50  0000 L CNN
 F 1 "Screw_Terminal_01x03" H 5980 2251 50  0000 L CNN
 F 2 "" H 5900 2300 50  0001 C CNN
