File: Diseño PCB/PCB-ESP32S/ModuloReles.sch (KiCad schematic (older format))
At the start: 8 parts, among them J1 Screw_Terminal_01x03, K1 SRD-05VDC-SL-C, Q1 MMBT2222A, U3 PC817

Commit message: Actualización Relé
Parts:
- added D?: 1N4007, Diode_THT:D_DO-41_SOD81_P10.16mm_Horizontal, symbol Diode:1N4007
- added D?: LED, symbol Device:LED
- added J?: Screw_Terminal_01x03, symbol Connector:Screw_Terminal_01x03
- added K?: SRD-05VDC-SL-C, RELAY_SRD-05VDC-SL-C, symbol Rele12V:SRD-05VDC-SL-C
- added Q?: MMBT2222A, SOT23, symbol MMBT2222A:MMBT2222A
- added R? (x2): R, symbol Device:R
- added U?: PC817, Package_DIP:DIP-4_W7.62mm, symbol Isolator:PC817
Connections:
- net labels added: IN2
- wire segments 23 -> 46
Changed lines of the file:
@@
 Text HLabel 1600 3150 0    50   Input ~ 0
 IN1
+$Comp
+L Diode:1N4007 D?
+U 1 1 61A9BBC4
+P 4250 4200
+F 0 "D?" V 4204 4280 50  0000 L CNN
+F 1 "1N4007" V 4295 4280 50  0000 L CNN
+F 2 "Diode_THT:D_DO-41_SOD81_P10.16mm_Horizontal" H 4250 4025 50  0001 C CNN
+F 3 "http://www.vishay.com/docs/88503/1n4001.pdf" H 4250 4200 50  0001 C CNN
+	1    4250 4200
+	0    1    1    0
+$EndComp
+$Comp
+L MMBT2222A:MMBT2222A Q?
+U 1 1 61A9BBCC
+P 4150 4900
+F 0 "Q?" H 4294 4946 50  0000 L CNN
+F 1 "MMBT2222A" H 4294 4855 50  0000 L CNN
+F 2 "SOT23" H 4150 4900 50  0001 L BNN
+F 3 "" H 4150 4900 50  0001 L BNN
+F 4 "568-4509-6-ND" H 4150 4900 50  0001 L BNN "DIGIKEY"
+F 5 "1757934" H 4150 4900 50  0001 L BNN "ELEMENT14"
+	1    4150 4900
+	1    0    0    -1
+$EndComp
+$Comp
+L Rele12V:SRD-05VDC-SL-C K?
+U 1 1 61A9BBD4
+P 4900 4150
+F 0 "K?" H 4900 4517 50  0000 C CNN
+F 1 "SRD-05VDC-SL-C" H 4900 4426 50  0000 C CNN
+F 2 "RELAY_SRD-05VDC-SL-C" H 4900 4150 50  0001 L BNN
+F 3 "" H 4900 4150 50  0001 L BNN
+F 4 "IPC-7251" H 4900 4150 50  0001 L BNN "STANDARD"
+F 5 "SONGLE RELAY" H 4900 4150 50  0001 L BNN "MANUFACTURER"
+	1    4900 4150
+	1    0    0    -1
+$EndComp
+$Comp
+L Connector:Screw_Terminal_01x03 J?
+U 1 1 61A9BBDA
+P 5900 4050
+F 0 "J?" H 5980 4092 50  0000 L CNN
+F 1 "Screw_Terminal_01x03" H 5980 4001 50  0000 L CNN
+F 2 "" H 5900 4050 50  0001 C CNN
+F 3 "~" H 5900 4050 50  0001 C CNN
+	1    5900 4050
+	1    0    0    -1
+$EndComp
+Wire Wire Line
+	4250 4050 4600 4050
+Wire Wire Line
+	4600 4350 4250 4350
+Wire Wire Line
+	4250 4350 4250 4700
+Connection ~ 4250 4350
+Wire Wire Line
+	4250 4050 3300 4050
+Connection ~ 4250 4050
+Wire Wire Line
+	5700 3950 5350 3950
+Wire Wire Line
+	5350 3950 5350 4050
+Wire Wire Line
+	5350 4050 5200 4050
+Wire Wire Line
+	5200 4150 5500 4150
+Wire Wire Line
+	5500 4150 5500 4050
+Wire Wire Line
+	5500 4050 5700 4050
+Wire Wire Line
+	5700 4150 5650 4150
+Wire Wire Line
+	5650 4150 5650 4350
+Wire Wire Line
+	5650 4350 5200 4350
+Text Label 5450 3950 0    50   ~ 0
+NO
+Text Label 5400 4150 0    50   ~ 0
+C
+Text Label 5400 4350 0    50   ~ 0
+NC
+Text HLabel 4250 5100 3    50   Input ~ 0
+GND
+$Comp
+L Device:R R?
+U 1 1 61AA55FC
+P 3650 4900
+F 0 "R?" H 3720 4946 50  0000 L CNN
+F 1 "R" H 3720 4855 50  0000 L CNN
+F 2 "" V 3580 4900 50  0001 C CNN
+F 3 "~" H 3650 4900 50  0001 C CNN
+	1    3650 4900
+	0    -1   -1   0
+$EndComp
+$Comp
+L Isolator:PC817 U?
+U 1 1 61AA5602
+P 2900 4800
+F 0 "U?" H 2900 5125 50  0000 C CNN
+F 1 "PC817" H 2900 5034 50  0000 C CNN
+F 2 "Package_DIP:DIP-4_W7.62mm" H 2700 4600 50  0001 L CIN
+F 3 "http://www.soselectronic.cz/a_info/resource/d/pc817.pdf" H 2900 4800 50  0001 L CNN
+	1    2900 4800
+	1    0    0    -1
+$EndComp
+$Comp
+L Device:LED D?
+U 1 1 61AA5608
+P 2000 4900
+F 0 "D?" H 1993 5117 50  0000 C CNN
+F 1 "LED" H 1993 5026 50  0000 C CNN
+F 2 "" H 2000 4900 50  0001 C CNN
+F 3 "~" H 2000 4900 50  0001 C CNN
+	1    2000 4900
+	1    0    0    -1
+$EndComp
+$Comp
+L Device:R R?
+U 1 1 61AA560E
+P 2300 4100
+F 0 "R?" H 2370 4146 50  0000 L CNN
+F 1 "R" H 2370 4055 50  0000 L CNN
+F 2 "" V 2230 4100 50  0001 C CNN
+F 3 "~" H 2300 4100 50  0001 C CNN
+	1    2300 4100
+	1    0    0    -1
+$EndComp
+Wire Wire Line
+	4050 4900 3800 4900
+Wire Wire Line
+	3500 4900 3200 4900
+Wire Wire Line
+	3300 4700 3200 4700
+Wire Wire Line
+	2600 4700 2300 4700
+Wire Wire Line
+	2300 4700 2300 4250
+Wire Wire Line
+	2300 3950 2300 3750
+Wire Wire Line
+	2600 4900 2150 4900
+Wire Wire Line
+	1850 4900 1600 4900
+Text HLabel 1600 4900 0    50   Input ~ 0
+IN2
+Wire Wire Line
+	3300 3750 3300 4050
+Connection ~ 3300 4050
+Wire Wire Line
+	3300 4050 3300 4700
+Text HLabel 2300 3700 1    50   Input ~ 0
+VESP32
+Text HLabel 3300 3750 1    50   Input ~ 0
+VCC_source
 $EndSCHEMATC

Commit message: Actualización footprints
Parts:
- D2, D?: footprint Diode_THT:D_DO-41_SOD81_P10.16mm_Horizontal -> Diode_SMD:D_SMA
- J1, J?: footprint (none) -> TerminalBlock:TerminalBlock_bornier-3_P5.08mm
Changed lines of the file:
@@
 F 0 "D2" V 4204 2530 50  0000 L CNN
 F 1 "1N4007" V 4295 2530 50  0000 L CNN
-F 2 "Diode_THT:D_DO-41_SOD81_P10.16mm_Horizontal" H 4250 2275 50  0001 C CNN
+F 2 "Diode_SMD:D_SMA" H 4250 2275 50  0001 C CNN
 F 3 "http://www.vishay.com/docs/88503/1n4001.pdf" H 4250 2450 50  0001 C CNN
 	1    4250 2450
@@
 F 0 "J1" H 5980 2342 50  0000 L CNN
 F 1 "Screw_Terminal_01x03" H 5980 2251 50  0000 L CNN
-F 2 "" H 5900 2300 50  0001 C CNN
+F 2 "TerminalBlock:TerminalBlock_bornier-3_P5.08mm" H 5900 2300 50  0001 C CNN
 F 3 "~" H 5900 2300 50  0001 C CNN
 	1    5900 2300
@@
 F 0 "D?" V 4204 4280 50  0000 L CNN
 F 1 "1N4007" V 4295 4280 50  0000 L CNN
-F 2 "Diode_THT:D_DO-41_SOD81_P10.16mm_Horizontal" H 4250 4025 50  0001 C CNN
+F 2 "Diode_SMD:D_SMA" H 4250 4025 50  0001 C CNN
 F 3 "http://www.vishay.com/docs/88503/1n4001.pdf" H 4250 4200 50  0001 C CNN
 	1    4250 4200
@@
 F 0 "J?" H 5980 4092 50  0000 L CNN
 F 1 "Screw_Terminal_01x03" H 5980 4001 50  0000 L CNN
-F 2 "" H 5900 4050 50  0001 C CNN
+F 2 "TerminalBlock:TerminalBlock_bornier-3_P5.08mm" H 5900 4050 50  0001 C CNN
 F 3 "~" H 5900 4050 50  0001 C CNN
 	1    5900 4050
