File: Diseño PCB/PCB-ESP32S/ModuloReles.sch (KiCad schematic (older format))
At the start: 16 parts, among them J1 Screw_Terminal_01x03, K1 SRD-05VDC-SL-C, Q1 MMBT2222A, U3 PC817

Commit message: esp-32 actualizacion
Parts:
- D1: footprint (none) -> LED_SMD:LED_0805_2012Metric_Pad1.15x1.40mm_HandSolder
- D2: footprint Diode_SMD:D_SMA -> Diode_SMD:D_SMA_Handsoldering
- D3: renamed from D?; footprint (none) -> LED_SMD:LED_0805_2012Metric_Pad1.15x1.40mm_HandSolder
- D4: renamed from D?; footprint Diode_SMD:D_SMA -> Diode_SMD:D_SMA_Handsoldering
- K1: footprint RELAY_SRD-05VDC-SL-C -> (none)
- K2: renamed from K?; footprint RELAY_SRD-05VDC-SL-C -> (none)
- Q1: footprint SOT23 -> (none)
- Q2: renamed from Q?; footprint SOT23 -> (none)
- R11, R4: renamed from R?; footprint (none) -> Resistor_SMD:R_0805_2012Metric_Pad1.20x1.40mm_HandSolder
- R5, R6: footprint (none) -> Resistor_SMD:R_0805_2012Metric_Pad1.20x1.40mm_HandSolder
- gave numbers to parts that had none: 2
Changed lines of the file:
@@
 $Descr A4 11693 8268
 encoding utf-8
-Sheet 4 8
+Sheet 3 8
 Title ""
 Date ""
@@
 F 0 "R6" H 3720 3196 50  0000 L CNN
 F 1 "R" H 3720 3105 50  0000 L CNN
-F 2 "" V 3580 3150 50  0001 C CNN
+F 2 "Resistor_SMD:R_0805_2012Metric_Pad1.20x1.40mm_HandSolder" V 3580 3150 50  0001 C CNN
 F 3 "~" H 3650 3150 50  0001 C CNN
 	1    3650 3150
@@
 F 0 "D2" V 4204 2530 50  0000 L CNN
 F 1 "1N4007" V 4295 2530 50  0000 L CNN
-F 2 "Diode_SMD:D_SMA" H 4250 2275 50  0001 C CNN
+F 2 "Diode_SMD:D_SMA_Handsoldering" H 4250 2275 50  0001 C CNN
 F 3 "http://www.vishay.com/docs/88503/1n4001.pdf" H 4250 2450 50  0001 C CNN
 	1    4250 2450
@@
 F 0 "Q1" H 4294 3196 50  0000 L CNN
 F 1 "MMBT2222A" H 4294 3105 50  0000 L CNN
-F 2 "SOT23" H 4150 3150 50  0001 L BNN
+F 2 "" H 4150 3150 50  0001 L BNN
 F 3 "" H 4150 3150 50  0001 L BNN
 F 4 "568-4509-6-ND" H 4150 3150 50  0001 L BNN "DIGIKEY"
@@
 F 0 "K1" H 4900 2767 50  0000 C CNN
 F 1 "SRD-05VDC-SL-C" H 4900 2676 50  0000 C CNN
-F 2 "RELAY_SRD-05VDC-SL-C" H 4900 2400 50  0001 L BNN
+F 2 "" H 4900 2400 50  0001 L BNN
 F 3 "" H 4900 2400 50  0001 L BNN
 F 4 "IPC-7251" H 4900 2400 50  0001 L BNN "STANDARD"
@@
 F 0 "D1" H 1993 3367 50  0000 C CNN
 F 1 "LED" H 1993 3276 50  0000 C CNN
-F 2 "" H 2000 3150 50  0001 C CNN
+F 2 "LED_SMD:LED_0805_2012Metric_Pad1.15x1.40mm_HandSolder" H 2000 3150 50  0001 C CNN
 F 3 "~" H 2000 3150 50  0001 C CNN
 	1    2000 3150
@@
 F 0 "R5" H 2370 2396 50  0000 L CNN
 F 1 "R" H 2370 2305 50  0000 L CNN
-F 2 "" V 2230 2350 50  0001 C CNN
+F 2 "Resistor_SMD:R_0805_2012Metric_Pad1.20x1.40mm_HandSolder" V 2230 2350 50  0001 C CNN
 F 3 "~" H 2300 2350 50  0001 C CNN
 	1    2300 2350
@@
 IN1
 $Comp
-L Diode:1N4007 D?
+L Diode:1N4007 D4
 U 1 1 61A9BBC4
 P 4250 4200
-F 0 "D?" V 4204 4280 50  0000 L CNN
+F 0 "D4" V 4204 4280 50  0000 L CNN
 F 1 "1N4007" V 4295 4280 50  0000 L CNN
-F 2 "Diode_SMD:D_SMA" H 4250 4025 50  0001 C CNN
+F 2 "Diode_SMD:D_SMA_Handsoldering" H 4250 4025 50  0001 C CNN
 F 3 "http://www.vishay.com/docs/88503/1n4001.pdf" H 4250 4200 50  0001 C CNN
 	1    4250 4200
@@
 $EndComp
 $Comp
-L MMBT2222A:MMBT2222A Q?
+L MMBT2222A:MMBT2222A Q2
 U 1 1 61A9BBCC
 P 4150 4900
-F 0 "Q?" H 4294 4946 50  0000 L CNN
+F 0 "Q2" H 4294 4946 50  0000 L CNN
 F 1 "MMBT2222A" H 4294 4855 50  0000 L CNN
-F 2 "SOT23" H 4150 4900 50  0001 L BNN
+F 2 "" H 4150 4900 50  0001 L BNN
 F 3 "" H 4150 4900 50  0001 L BNN
 F 4 "568-4509-6-ND" H 4150 4900 50  0001 L BNN "DIGIKEY"
@@
 $EndComp
 $Comp
-L Rele12V:SRD-05VDC-SL-C K?
+L Rele12V:SRD-05VDC-SL-C K2
 U 1 1 61A9BBD4
 P 4900 4150
-F 0 "K?" H 4900 4517 50  0000 C CNN
+F 0 "K2" H 4900 4517 50  0000 C CNN
 F 1 "SRD-05VDC-SL-C" H 4900 4426 50  0000 C CNN
-F 2 "RELAY_SRD-05VDC-SL-C" H 4900 4150 50  0001 L BNN
+F 2 "" H 4900 4150 50  0001 L BNN
 F 3 "" H 4900 4150 50  0001 L BNN
 F 4 "IPC-7251" H 4900 4150 50  0001 L BNN "STANDARD"
@@
 $EndComp
 $Comp
-L Connector:Screw_Terminal_01x03 J?
+L Connector:Screw_Terminal_01x03 J3
 U 1 1 61A9BBDA
 P 5900 4050
-F 0 "J?" H 5980 4092 50  0000 L CNN
+F 0 "J3" H 5980 4092 50  0000 L CNN
 F 1 "Screw_Terminal_01x03" H 5980 4001 50  0000 L CNN
 F 2 "TerminalBlock:TerminalBlock_bornier-3_P5.08mm" H 5900 4050 50  0001 C CNN
@@
 GND
 $Comp
-L Device:R R?
+L Device:R R11
 U 1 1 61AA55FC
 P 3650 4900
-F 0 "R?" H 3720 4946 50  0000 L CNN
+F 0 "R11" H 3720 4946 50  0000 L CNN
 F 1 "R" H 3720 4855 50  0000 L CNN
-F 2 "" V 3580 4900 50  0001 C CNN
+F 2 "Resistor_SMD:R_0805_2012Metric_Pad1.20x1.40mm_HandSolder" V 3580 4900 50  0001 C CNN
 F 3 "~" H 3650 4900 50  0001 C CNN
 	1    3650 4900
@@
 $EndComp
 $Comp
-L Isolator:PC817 U?
+L Isolator:PC817 U4
 U 1 1 61AA5602
 P 2900 4800
-F 0 "U?" H 2900 5125 50  0000 C CNN
+F 0 "U4" H 2900 5125 50  0000 C CNN
 F 1 "PC817" H 2900 5034 50  0000 C CNN
 F 2 "Package_DIP:DIP-4_W7.62mm" H 2700 4600 50  0001 L CIN
@@
 $EndComp
 $Comp
-L Device:LED D?
+L Device:LED D3
 U 1 1 61AA5608
 P 2000 4900
-F 0 "D?" H 1993 5117 50  0000 C CNN
+F 0 "D3" H 1993 5117 50  0000 C CNN
 F 1 "LED" H 1993 5026 50  0000 C CNN
-F 2 "" H 2000 4900 50  0001 C CNN
+F 2 "LED_SMD:LED_0805_2012Metric_Pad1.15x1.40mm_HandSolder" H 2000 4900 50  0001 C CNN
 F 3 "~" H 2000 4900 50  0001 C CNN
 	1    2000 4900
@@
 $EndComp
 $Comp
-L Device:R R?
+L Device:R R4
 U 1 1 61AA560E
 P 2300 4100
-F 0 "R?" H 2370 4146 50  0000 L CNN
+F 0 "R4" H 2370 4146 50  0000 L CNN
 F 1 "R" H 2370 4055 50  0000 L CNN
-F 2 "" V 2230 4100 50  0001 C CNN
+F 2 "Resistor_SMD:R_0805_2012Metric_Pad1.20x1.40mm_HandSolder" V 2230 4100 50  0001 C CNN
 F 3 "~" H 2300 4100 50  0001 C CNN
 	1    2300 4100

Commit message: .
Parts:
- K1, K2: symbol Rele12V:SRD-05VDC-SL-C -> PCB-ESP32S-rescue:SRD-05VDC-SL-C-Rele12V
- Q1, Q2: symbol MMBT2222A:MMBT2222A -> PCB-ESP32S-rescue:MMBT2222A-MMBT2222A
Changed lines of the file:
@@
 $EndComp
 $Comp
-L MMBT2222A:MMBT2222A Q1
+L PCB-ESP32S-rescue:MMBT2222A-MMBT2222A Q1
 U 1 1 61A825BF
 P 4150 3150
@@
 $EndComp
 $Comp
-L Rele12V:SRD-05VDC-SL-C K1
+L PCB-ESP32S-rescue:SRD-05VDC-SL-C-Rele12V K1
 U 1 1 61A82FC5
 P 4900 2400
@@
 $EndComp
 $Comp
-L MMBT2222A:MMBT2222A Q2
+L PCB-ESP32S-rescue:MMBT2222A-MMBT2222A Q2
 U 1 1 61A9BBCC
 P 4150 4900
@@
 $EndComp
 $Comp
-L Rele12V:SRD-05VDC-SL-C K2
+L PCB-ESP32S-rescue:SRD-05VDC-SL-C-Rele12V K2
 U 1 1 61A9BBD4
 P 4900 4150

Commit message: Actualización footprints
Parts:
- K1, K2: footprint (none) -> ModuloRele:RELAY_SRD-05VDC-SL-C; symbol PCB-ESP32S-rescue:SRD-05VDC-SL-C-Rele12V -> PCB-ESP32S-rescue:SRD-05VDC-SL-C-Rele12V-PCB-ESP32S-rescue
- Q1, Q2: footprint (none) -> ModuloRele:SOT23; symbol PCB-ESP32S-rescue:MMBT2222A-MMBT2222A -> PCB-ESP32S-rescue:MMBT2222A-MMBT2222A-PCB-ESP32S-rescue
Connections:
- net IN1 renamed GPIO1
- net IN2 renamed GPIO2
Changed lines of the file:
@@
 $EndComp
 $Comp
-L PCB-ESP32S-rescue:MMBT2222A-MMBT2222A Q1
+L PCB-ESP32S-rescue:MMBT2222A-MMBT2222A-PCB-ESP32S-rescue Q1
 U 1 1 61A825BF
 P 4150 3150
 F 0 "Q1" H 4294 3196 50  0000 L CNN
 F 1 "MMBT2222A" H 4294 3105 50  0000 L CNN
-F 2 "" H 4150 3150 50  0001 L BNN
+F 2 "ModuloRele:SOT23" H 4150 3150 50  0001 L BNN
 F 3 "" H 4150 3150 50  0001 L BNN
 F 4 "568-4509-6-ND" H 4150 3150 50  0001 L BNN "DIGIKEY"
@@
 $EndComp
 $Comp
-L PCB-ESP32S-rescue:SRD-05VDC-SL-C-Rele12V K1
+L PCB-ESP32S-rescue:SRD-05VDC-SL-C-Rele12V-PCB-ESP32S-rescue K1
 U 1 1 61A82FC5
 P 4900 2400
 F 0 "K1" H 4900 2767 50  0000 C CNN
 F 1 "SRD-05VDC-SL-C" H 4900 2676 50  0000 C CNN
-F 2 "" H 4900 2400 50  0001 L BNN
+F 2 "ModuloRele:RELAY_SRD-05VDC-SL-C" H 4900 2400 50  0001 L BNN
 F 3 "" H 4900 2400 50  0001 L BNN
 F 4 "IPC-7251" H 4900 2400 50  0001 L BNN "STANDARD"
@@
 GND
 Text HLabel 1600 3150 0    50   Input ~ 0
-IN1
+GPIO1
 $Comp
 L Diode:1N4007 D4
@@
 $EndComp
 $Comp
-L PCB-ESP32S-rescue:MMBT2222A-MMBT2222A Q2
+L PCB-ESP32S-rescue:MMBT2222A-MMBT2222A-PCB-ESP32S-rescue Q2
 U 1 1 61A9BBCC
 P 4150 4900
 F 0 "Q2" H 4294 4946 50  0000 L CNN
 F 1 "MMBT2222A" H 4294 4855 50  0000 L CNN
-F 2 "" H 4150 4900 50  0001 L BNN
+F 2 "ModuloRele:SOT23" H 4150 4900 50  0001 L BNN
 F 3 "" H 4150 4900 50  0001 L BNN
 F 4 "568-4509-6-ND" H 4150 4900 50  0001 L BNN "DIGIKEY"
@@
 $EndComp
 $Comp
-L PCB-ESP32S-rescue:SRD-05VDC-SL-C-Rele12V K2
+L PCB-ESP32S-rescue:SRD-05VDC-SL-C-Rele12V-PCB-ESP32S-rescue K2
 U 1 1 61A9BBD4
 P 4900 4150
 F 0 "K2" H 4900 4517 50  0000 C CNN
 F 1 "SRD-05VDC-SL-C" H 4900 4426 50  0000 C CNN
-F 2 "" H 4900 4150 50  0001 L BNN
+F 2 "ModuloRele:RELAY_SRD-05VDC-SL-C" H 4900 4150 50  0001 L BNN
 F 3 "" H 4900 4150 50  0001 L BNN
 F 4 "IPC-7251" H 4900 4150 50  0001 L BNN "STANDARD"
@@
 	1850 4900 1600 4900
 Text HLabel 1600 4900 0    50   Input ~ 0
-IN2
+GPIO2
 Wire Wire Line
 	3300 3750 3300 4050
