File: Diseño PCB/PCB-ESP32S/pines_sensor.sch (KiCad schematic (older format))
At the start: 1 part

Commit message: Humedad y luz
Parts:
- gave numbers to parts that had none: 1
Changed lines of the file:
@@
 $Descr A4 11693 8268
 encoding utf-8
-Sheet 3 4
+Sheet 3 5
 Title ""
 Date ""
@@
 $EndDescr
 $Comp
-L pines_yl100&mq135:pines_sensor U?
+L pines_yl100&mq135:pines_sensor U2
 U 1 1 619FDFBF
 P 3050 2350
-F 0 "U?" H 3428 2338 50  0000 L CNN
+F 0 "U2" H 3428 2338 50  0000 L CNN
 F 1 "pines_sensor" H 3428 2247 50  0000 L CNN
 F 2 "" H 3050 2350 50  0001 C CNN
