File: Diseño PCB/PCB-ESP32S/pines_sensor.sch (KiCad schematic (older format))
At the start: 1 part, among them U2 pines_sensor

Commit message: .
Parts:
- U2: symbol pines_yl100&mq135:pines_sensor -> PCB-ESP32S-rescue:pines_sensor-pines_yl100&mq135
Changed lines of the file:
@@
 $EndDescr
 $Comp
-L pines_yl100&mq135:pines_sensor U2
+L PCB-ESP32S-rescue:pines_sensor-pines_yl100&mq135 U2
 U 1 1 619FDFBF
 P 3050 2350

Commit message: Actualización footprints
Parts:
- U2: symbol PCB-ESP32S-rescue:pines_sensor-pines_yl100&mq135 -> PCB-ESP32S-rescue:pines_sensor-pines_yl100&mq135-PCB-ESP32S-rescue
Changed lines of the file:
@@
 $EndDescr
 $Comp
-L PCB-ESP32S-rescue:pines_sensor-pines_yl100&mq135 U2
+L PCB-ESP32S-rescue:pines_sensor-pines_yl100&mq135-PCB-ESP32S-rescue U2
 U 1 1 619FDFBF
 P 3050 2350
