File: Diseño PCB/PCB-ESP32S/PCB-ESP32S.sch (KiCad schematic (older format))
At the start: 5 parts, among them SW1 SW_DIP_x01, SW2 SW_DIP_x01, U1 ESP-32S

Commit message: esp-32 actualizacion
Parts:
- added D10, D9: LED, symbol Device:LED
- added J7: Screw_Terminal_01x03, TerminalBlock:TerminalBlock_bornier-3_P5.08mm, symbol Connector:Screw_Terminal_01x03
- added R16, R17: 220, Resistor_SMD:R_0805_2012Metric_Pad1.20x1.40mm_HandSolder, symbol Device:R
- R1, R2: footprint Resistor_SMD:R_0603_1608Metric -> Resistor_SMD:R_0805_2012Metric_Pad1.20x1.40mm_HandSolder
Connections:
- wire segments 33 -> 55

Commit message: .
Parts:
- U1: symbol PCB-ESP32S-rescue:ESP-32S-ESP32S -> PCB-ESP32S-rescue:ESP-32S-ESP32S-PCB-ESP32S-rescue
Changed lines of the file:
@@
 F6 "ADDR" I R 9150 2700 50
 $EndSheet
-$Comp
-L power:+5V #PWR0109
-U 1 1 61A9FC1E
-P 8300 2450
-F 0 "#PWR0109" H 8300 2300 50  0001 C CNN
-F 1 "+5V" H 8315 2623 50  0000 C CNN
-F 2 "" H 8300 2450 50  0001 C CNN
-F 3 "" H 8300 2450 50  0001 C CNN
-	1    8300 2450
-	1    0    0    -1
-$EndComp
 Wire Wire Line
 	8550 2500 8300 2500
@@
 $EndComp
 $Comp
-L PCB-ESP32S-rescue:ESP-32S-ESP32S U1
+L PCB-ESP32S-rescue:ESP-32S-ESP32S-PCB-ESP32S-rescue U1
 U 1 1 619F8438
 P 5100 3800
@@
 Wire Wire Line
 	4650 4850 4650 5200
+$Comp
+L power:+3.3V #PWR?
+U 1 1 61BACFBA
+P 8300 2450
+F 0 "#PWR?" H 8300 2300 50  0001 C CNN
+F 1 "+3.3V" H 8315 2623 50  0000 C CNN
+F 2 "" H 8300 2450 50  0001 C CNN
+F 3 "" H 8300 2450 50  0001 C CNN
+	1    8300 2450
+	1    0    0    -1
+$EndComp
 $EndSCHEMATC

Commit message: Actualización footprints
Parts:
- U1: symbol PCB-ESP32S-rescue:ESP-32S-ESP32S-PCB-ESP32S-rescue -> PCB-ESP32S-rescue:ESP-32S-ESP32S-PCB-ESP32S-rescue-PCB-ESP32S-rescue
Changed lines of the file:
@@
 $EndComp
 $Comp
-L PCB-ESP32S-rescue:ESP-32S-ESP32S-PCB-ESP32S-rescue U1
+L PCB-ESP32S-rescue:ESP-32S-ESP32S-PCB-ESP32S-rescue-PCB-ESP32S-rescue U1
 U 1 1 619F8438
 P 5100 3800

Commit message: Actualización
Changed lines of the file:
@@
 $Descr A4 11693 8268
 encoding utf-8
-Sheet 1 8
+Sheet 1 7
 Title ""
 Date ""
@@
 	8300 2600 8300 2650
 $Sheet
-S 4500 5450 850  850
-U 61A8D74F
-F0 "Sheet61A8D74E" 50
-F1 "12volts.sch" 50
-F2 "GND" I R 5350 6050 50
-F3 "12V" I R 5350 5700 50
-F4 "AC1" I L 4500 5700 50
-F5 "AC2" I L 4500 6050 50
-$EndSheet
-$Sheet
-S 2000 5000 1500 1400
+S 2100 5000 1500 1400
 U 61A8C81F
 F0 "Sheet61A8C81E" 50
 F1 "alimentacion.sch" 50
-F2 "5V" I R 3500 5650 50
-F3 "12V" I L 2000 5350 50
-F4 "3.3V" I R 3500 5850 50
-F5 "GND" I L 2000 6000 50
+F2 "5V" I R 3600 5650 50
+F3 "12V" I L 2100 5350 50
+F4 "3.3V" I R 3600 5850 50
+F5 "GND" I L 2100 6000 50
 $EndSheet
 $Sheet
