File: Diseño PCB/PCB-ESP32S/PCB-ESP32S.sch (KiCad schematic (older format))
At the start: 10 parts, among them J7 Screw_Terminal_01x03, SW1 SW_DIP_x01, SW2 SW_DIP_x01, U1 ESP-32S

Commit message: verificacion componentes
Parts:
- D10, D9: footprint (none) -> LED_SMD:LED_0805_2012Metric_Pad1.15x1.40mm_HandSolder
Changed lines of the file:
@@
 F 0 "D10" H 6093 4867 50  0000 C CNN
 F 1 "LED" H 6093 4776 50  0000 C CNN
-F 2 "" H 6100 4650 50  0001 C CNN
+F 2 "LED_SMD:LED_0805_2012Metric_Pad1.15x1.40mm_HandSolder" H 6100 4650 50  0001 C CNN
 F 3 "~" H 6100 4650 50  0001 C CNN
 	1    6100 4650
@@
 F 0 "D9" H 2243 2967 50  0000 C CNN
 F 1 "LED" H 2243 2876 50  0000 C CNN
-F 2 "" H 2250 2750 50  0001 C CNN
+F 2 "LED_SMD:LED_0805_2012Metric_Pad1.15x1.40mm_HandSolder" H 2250 2750 50  0001 C CNN
 F 3 "~" H 2250 2750 50  0001 C CNN
 	1    2250 2750
@@
 	4650 4850 4650 5200
 $Comp
-L power:+3.3V #PWR?
+L power:+3.3V #PWR0109
 U 1 1 61BACFBA
 P 8300 2450
-F 0 "#PWR?" H 8300 2300 50  0001 C CNN
+F 0 "#PWR0109" H 8300 2300 50  0001 C CNN
 F 1 "+3.3V" H 8315 2623 50  0000 C CNN
 F 2 "" H 8300 2450 50  0001 C CNN
@@
 F7 "OUT-" I R 6950 1700 50
 $EndSheet
+$Comp
+L power:+5V #PWR?
+U 1 1 61BFAAB8
+P 7500 4750
+F 0 "#PWR?" H 7500 4600 50  0001 C CNN
+F 1 "+5V" H 7515 4923 50  0000 C CNN
+F 2 "" H 7500 4750 50  0001 C CNN
+F 3 "" H 7500 4750 50  0001 C CNN
+	1    7500 4750
+	1    0    0    -1
+$EndComp
+$Comp
+L power:+5V #PWR?
+U 1 1 61BFB043
+P 9000 4750
+F 0 "#PWR?" H 9000 4600 50  0001 C CNN
+F 1 "+5V" H 9015 4923 50  0000 C CNN
+F 2 "" H 9000 4750 50  0001 C CNN
+F 3 "" H 9000 4750 50  0001 C CNN
+	1    9000 4750
+	1    0    0    -1
+$EndComp
+$Comp
+L power:+5V #PWR?
+U 1 1 61BFB68C
+P 3750 5600
+F 0 "#PWR?" H 3750 5450 50  0001 C CNN
+F 1 "+5V" H 3765 5773 50  0000 C CNN
+F 2 "" H 3750 5600 50  0001 C CNN
+F 3 "" H 3750 5600 50  0001 C CNN
+	1    3750 5600
+	1    0    0    -1
+$EndComp
+$Comp
+L power:+3.3V #PWR?
+U 1 1 61BFBED1
+P 3750 5800
+F 0 "#PWR?" H 3750 5650 50  0001 C CNN
+F 1 "+3.3V" H 3765 5973 50  0000 C CNN
+F 2 "" H 3750 5800 50  0001 C CNN
+F 3 "" H 3750 5800 50  0001 C CNN
+	1    3750 5800
+	1    0    0    -1
+$EndComp
+Wire Wire Line
+	3600 5650 3750 5650
+Wire Wire Line
+	3750 5650 3750 5600
+Wire Wire Line
+	3600 5850 3750 5850
+Wire Wire Line
+	3750 5850 3750 5800
+Wire Wire Line
+	7700 4800 7500 4800
+Wire Wire Line
+	7500 4800 7500 4750
+Wire Wire Line
+	9200 4800 9000 4800
+Wire Wire Line
+	9000 4800 9000 4750
+$Comp
+L power:GND #PWR?
+U 1 1 61C011C0
+P 7550 5350
+F 0 "#PWR?" H 7550 5100 50  0001 C CNN
+F 1 "GND" H 7555 5177 50  0000 C CNN
+F 2 "" H 7550 5350 50  0001 C CNN
+F 3 "" H 7550 5350 50  0001 C CNN
+	1    7550 5350
+	1    0    0    -1
+$EndComp
+$Comp
+L power:GND #PWR?
+U 1 1 61C01E8D
+P 1900 6100
+F 0 "#PWR?" H 1900 5850 50  0001 C CNN
+F 1 "GND" H 1905 5927 50  0000 C CNN
+F 2 "" H 1900 6100 50  0001 C CNN
+F 3 "" H 1900 6100 50  0001 C CNN
+	1    1900 6100
+	1    0    0    -1
+$EndComp
+$Comp
+L power:GND #PWR?
+U 1 1 61C0250D
+P 9050 5450
+F 0 "#PWR?" H 9050 5200 50  0001 C CNN
+F 1 "GND" H 9055 5277 50  0000 C CNN
+F 2 "" H 9050 5450 50  0001 C CNN
+F 3 "" H 9050 5450 50  0001 C CNN
+	1    9050 5450
+	1    0    0    -1
+$EndComp
+$Comp
+L power:GND #PWR?
+U 1 1 61C02BAF
+P 9350 3950
+F 0 "#PWR?" H 9350 3700 50  0001 C CNN
+F 1 "GND" H 9355 3777 50  0000 C CNN
+F 2 "" H 9350 3950 50  0001 C CNN
+F 3 "" H 9350 3950 50  0001 C CNN
+	1    9350 3950
+	1    0    0    -1
+$EndComp
+$Comp
+L power:GND #PWR?
+U 1 1 61C036E2
+P 5850 1950
+F 0 "#PWR?" H 5850 1700 50  0001 C CNN
+F 1 "GND" H 5855 1777 50  0000 C CNN
+F 2 "" H 5850 1950 50  0001 C CNN
+F 3 "" H 5850 1950 50  0001 C CNN
+	1    5850 1950
+	1    0    0    -1
+$EndComp
+$Comp
+L power:GND #PWR?
+U 1 1 61C03D07
+P 7500 1750
+F 0 "#PWR?" H 7500 1500 50  0001 C CNN
+F 1 "GND" H 7505 1577 50  0000 C CNN
+F 2 "" H 7500 1750 50  0001 C CNN
+F 3 "" H 7500 1750 50  0001 C CNN
+	1    7500 1750
+	1    0    0    -1
+$EndComp
+Wire Wire Line
+	6100 1900 5850 1900
+Wire Wire Line
+	5850 1900 5850 1950
+Wire Wire Line
+	7500 1750 7500 1700
+Wire Wire Line
+	7500 1700 6950 1700
 $EndSCHEMATC

Commit message: LuzSens-actualización
Connections:
- no-connect marks 0 -> 1
Changed lines of the file:
@@
 Wire Wire Line
 	7500 1700 6950 1700
+NoConn ~ 9150 2700
 $EndSCHEMATC

Commit message: Pines sensores
Connections:
- net IO14: now reaches U1.13 (IO14)
- net IO12: now reaches U1.14 (IO12)
- net IO2: now reaches U1.24 (IO2)
- net IO32: now reaches U1.8 (IO32)
- net IO33: now reaches U1.9 (IO33)
- net IO4: no longer names the net of U1.26 (IO4)
- no-connect marks 1 -> 3
Changed lines of the file:
@@
 	8150 3650 8400 3650
 Text GLabel 8150 3800 0    50   Input ~ 0
-IO4
+IO2
 Wire Wire Line
 	8150 3800 8400 3800
-Text GLabel 6050 4350 2    50   Input ~ 0
-IO4
-Wire Wire Line
-	6050 4350 6000 4350
 $Sheet
 S 9500 3400 750  600
@@
 $EndSheet
 $Sheet
-S 7700 4600 1050 800
+S 7700 4600 850  800
 U 619FC5E1
-F0 "Sheet619FC5E0" 50
+F0 "YL-100" 50
 F1 "pines_sensor.sch" 50
 F2 "VCC" I L 7700 4800 50
 F3 "GND" I L 7700 5300 50
-F4 "Aout" I R 8750 4800 50
-F5 "Dout" I R 8750 5300 50
+F4 "Aout" I R 8550 4800 50
+F5 "Dout" I R 8550 5300 50
 $EndSheet
 $Sheet
-S 9200 4600 1050 800
+S 9200 4600 850  800
 U 61A90AD5
-F0 "sheet61A90ACF" 50
+F0 "MQ-135" 50
 F1 "pines_sensor.sch" 50
 F2 "VCC" I L 9200 4800 50
 F3 "GND" I L 9200 5300 50
-F4 "Aout" I R 10250 4800 50
-F5 "Dout" I R 10250 5300 50
+F4 "Aout" I R 10050 4800 50
+F5 "Dout" I R 10050 5300 50
 $EndSheet
 Connection ~ 2800 2500
@@
 F 3 "" H 2800 2400 50  0001 C CNN
 	1    2800 2400
-	1    0    0    -1
-$EndComp
-$Comp
-L PCB-ESP32S-rescue:ESP-32S-ESP32S-PCB-ESP32S-rescue-PCB-ESP32S-rescue U1
-U 1 1 619F8438
-P 5100 3800
-F 0 "U1" H 5075 5187 60  0000 C CNN
-F 1 "ESP-32S" H 5075 5081 60  0000 C CNN
-F 2 "ESP32S:ESP-32S" H 5450 5150 60  0001 C CNN
-F 3 "" H 4650 4250 60  0001 C CNN
-	1    5100 3800
 	1    0    0    -1
 $EndComp
@@
 	7500 1700 6950 1700
 NoConn ~ 9150 2700
+$Comp
+L PCB-ESP32S-rescue:ESP-32S-ESP32S-PCB-ESP32S-rescue-PCB-ESP32S-rescue U1
+U 1 1 619F8438
+P 5100 3800
+F 0 "U1" H 5075 5187 60  0000 C CNN
+F 1 "ESP-32S" H 5075 5081 60  0000 C CNN
+F 2 "ESP32S:ESP-32S" H 5450 5150 60  0001 C CNN
+F 3 "" H 4650 4250 60  0001 C CNN
+	1    5100 3800
+	1    0    0    -1
+$EndComp
+Text GLabel 5650 4850 2    50   Input ~ 0
+IO2
+Wire Wire Line
+	5550 4850 5650 4850
+Text GLabel 8350 2950 0    50   Input ~ 0
+IO32
+Text GLabel 9500 2500 2    50   Input ~ 0
+IO33
+Wire Wire Line
+	9500 2500 9150 2500
+Wire Wire Line
+	8550 2700 8450 2700
+Wire Wire Line
+	8450 2700 8450 2950
+Wire Wire Line
+	8450 2950 8350 2950
+Text GLabel 3950 3800 0    50   Input ~ 0
+IO32
+Text GLabel 3950 3900 0    50   Input ~ 0
+IO33
+Wire Wire Line
+	3950 3800 4150 3800
+Wire Wire Line
+	3950 3900 4150 3900
+Text GLabel 8650 4800 2    50   Input ~ 0
+IO12
+Text GLabel 10150 4800 2    50   Input ~ 0
+IO14
+Wire Wire Line
+	10150 4800 10050 4800
+Wire Wire Line
+	8650 4800 8550 4800
+NoConn ~ 8550 5300
+NoConn ~ 10050 5300
+Text GLabel 3950 4400 0    50   Input ~ 0
+IO12
+Text GLabel 3950 4300 0    50   Input ~ 0
+IO14
+Wire Wire Line
+	3950 4300 4150 4300
+Wire Wire Line
+	3950 4400 4150 4400
+Wire Wire Line
+	9200 5300 9050 5300
+Wire Wire Line
+	9050 5300 9050 5450
+Wire Wire Line
+	7700 5300 7550 5300
+Wire Wire Line
+	7550 5300 7550 5350
+Wire Wire Line
+	9500 3850 9350 3850
+Wire Wire Line
+	9350 3850 9350 3950
+Wire Wire Line
+	2100 6000 1900 6000
+Wire Wire Line
+	1900 6000 1900 6100
 $EndSCHEMATC

Commit message: Baterías
Changed lines of the file:
@@
 $Descr A4 11693 8268
 encoding utf-8
-Sheet 1 8
+Sheet 1 7
 Title ""
 Date ""
@@
 	8300 2600 8300 2650
 $Sheet
-S 2100 5000 1500 1400
-U 61A8C81F
-F0 "Sheet61A8C81E" 50
-F1 "alimentacion.sch" 50
-F2 "5V" I R 3600 5650 50
-F3 "12V" I L 2100 5350 50
-F4 "3.3V" I R 3600 5850 50
-F5 "GND" I L 2100 6000 50
-$EndSheet
-$Sheet
 S 7700 4600 850  800
 U 619FC5E1
@@
 	1    0    0    -1
 $EndComp
-$Sheet
-S 6100 1400 850  750
-U 61BD2E90
-F0 "baterias" 50
-F1 "baterias.sch" 50
-F2 "IN+" I L 6100 1650 50
-F3 "IN-" I L 6100 1900 50
-F4 "OUT+" I R 6950 1550 50
-F5 "BAT+" I R 6950 1850 50
-F6 "BAT-" I R 6950 2000 50
-F7 "OUT-" I R 6950 1700 50
-$EndSheet
 $Comp
 L power:+5V #PWR?
@@
 	1    0    0    -1
 $EndComp
-$Comp
-L power:GND #PWR?
-U 1 1 61C036E2
-P 5850 1950
-F 0 "#PWR?" H 5850 1700 50  0001 C CNN
-F 1 "GND" H 5855 1777 50  0000 C CNN
-F 2 "" H 5850 1950 50  0001 C CNN
-F 3 "" H 5850 1950 50  0001 C CNN
-	1    5850 1950
-	1    0    0    -1
-$EndComp
-$Comp
-L power:GND #PWR?
-U 1 1 61C03D07
-P 7500 1750
-F 0 "#PWR?" H 7500 1500 50  0001 C CNN
-F 1 "GND" H 7505 1577 50  0000 C CNN
-F 2 "" H 7500 1750 50  0001 C CNN
-F 3 "" H 7500 1750 50  0001 C CNN
-	1    7500 1750
-	1    0    0    -1
-$EndComp
-Wire Wire Line
-	6100 1900 5850 1900
-Wire Wire Line
-	5850 1900 5850 1950
-Wire Wire Line
-	7500 1750 7500 1700
-Wire Wire Line
-	7500 1700 6950 1700
 NoConn ~ 9150 2700
 $Comp
@@
 Wire Wire Line
 	1900 6000 1900 6100
+$Sheet
+S 2100 5000 1500 1400
+U 61A8C81F
+F0 "Sheet61A8C81E" 50
+F1 "alimentacion.sch" 50
+F2 "5V" I R 3600 5650 50
+F3 "12V" I L 2100 5350 50
+F4 "3.3V" I R 3600 5850 50
+F5 "GND" I L 2100 6000 50
+$EndSheet
 $EndSCHEMATC

Commit message: separacion
Connections:
- no-connect marks 3 -> 2
Changed lines of the file:
@@
 $Descr A4 11693 8268
 encoding utf-8
-Sheet 1 7
+Sheet 1 6
 Title ""
 Date ""
@@
 Wire Wire Line
 	8150 3800 8400 3800
-$Sheet
-S 9500 3400 750  600
-U 61A61E97
-F0 "ModulosReles" 50
-F1 "ModuloReles.sch" 50
-F2 "VESP32" I L 9500 3550 50
-F3 "VCC_source" I L 9500 3700 50
-F4 "GND" I L 9500 3850 50
-F5 "IN1" I R 10250 3600 50
-F6 "IN2" I R 10250 3800 50
-$EndSheet
 $Sheet
 S 8550 2300 600  550
@@
 	8300 2600 8300 2650
 $Sheet
-S 7700 4600 850  800
-U 619FC5E1
-F0 "YL-100" 50
-F1 "pines_sensor.sch" 50
-F2 "VCC" I L 7700 4800 50
-F3 "GND" I L 7700 5300 50
-F4 "Aout" I R 8550 4800 50
-F5 "Dout" I R 8550 5300 50
-$EndSheet
-$Sheet
 S 9200 4600 850  800
 U 61A90AD5
@@
 F3 "GND" I L 9200 5300 50
 F4 "Aout" I R 10050 4800 50
-F5 "Dout" I R 10050 5300 50
 $EndSheet
 Connection ~ 2800 2500
@@
 $EndComp
 $Comp
-L power:+5V #PWR?
+L power:+5V #PWR0111
 U 1 1 61BFAAB8
 P 7500 4750
-F 0 "#PWR?" H 7500 4600 50  0001 C CNN
+F 0 "#PWR0111" H 7500 4600 50  0001 C CNN
 F 1 "+5V" H 7515 4923 50  0000 C CNN
 F 2 "" H 7500 4750 50  0001 C CNN
@@
 $EndComp
 $Comp
-L power:+5V #PWR?
+L power:+5V #PWR0112
 U 1 1 61BFB043
 P 9000 4750
-F 0 "#PWR?" H 9000 4600 50  0001 C CNN
+F 0 "#PWR0112" H 9000 4600 50  0001 C CNN
 F 1 "+5V" H 9015 4923 50  0000 C CNN
 F 2 "" H 9000 4750 50  0001 C CNN
@@
 $EndComp
 $Comp
-L power:+5V #PWR?
+L power:+5V #PWR0113
 U 1 1 61BFB68C
 P 3750 5600
-F 0 "#PWR?" H 3750 5450 50  0001 C CNN
+F 0 "#PWR0113" H 3750 5450 50  0001 C CNN
 F 1 "+5V" H 3765 5773 50  0000 C CNN
 F 2 "" H 3750 5600 50  0001 C CNN
@@
 $EndComp
 $Comp
-L power:+3.3V #PWR?
+L power:+3.3V #PWR0114
 U 1 1 61BFBED1
 P 3750 5800
-F 0 "#PWR?" H 3750 5650 50  0001 C CNN
+F 0 "#PWR0114" H 3750 5650 50  0001 C CNN
 F 1 "+3.3V" H 3765 5973 50  0000 C CNN
 F 2 "" H 3750 5800 50  0001 C CNN
@@
 	3750 5850 3750 5800
 Wire Wire Line
-	7700 4800 7500 4800
-Wire Wire Line
 	7500 4800 7500 4750
 Wire Wire Line
@@
 	9000 4800 9000 4750
 $Comp
-L power:GND #PWR?
+L power:GND #PWR0115
 U 1 1 61C011C0
 P 7550 5350
-F 0 "#PWR?" H 7550 5100 50  0001 C CNN
+F 0 "#PWR0115" H 7550 5100 50  0001 C CNN
 F 1 "GND" H 7555 5177 50  0000 C CNN
 F 2 "" H 7550 5350 50  0001 C CNN
@@
 $EndComp
 $Comp
-L power:GND #PWR?
+L power:GND #PWR0116
 U 1 1 61C01E8D
 P 1900 6100
-F 0 "#PWR?" H 1900 5850 50  0001 C CNN
+F 0 "#PWR0116" H 1900 5850 50  0001 C CNN
 F 1 "GND" H 1905 5927 50  0000 C CNN
 F 2 "" H 1900 6100 50  0001 C CNN
@@
 $EndComp
 $Comp
-L power:GND #PWR?
+L power:GND #PWR0117
 U 1 1 61C0250D
 P 9050 5450
-F 0 "#PWR?" H 9050 5200 50  0001 C CNN
+F 0 "#PWR0117" H 9050 5200 50  0001 C CNN
 F 1 "GND" H 9055 5277 50  0000 C CNN
 F 2 "" H 9050 5450 50  0001 C CNN
 F 3 "" H 9050 5450 50  0001 C CNN
 	1    9050 5450
-	1    0    0    -1
-$EndComp
-$Comp
-L power:GND #PWR?
-U 1 1 61C02BAF
-P 9350 3950
-F 0 "#PWR?" H 9350 3700 50  0001 C CNN
-F 1 "GND" H 9355 3777 50  0000 C CNN
-F 2 "" H 9350 3950 50  0001 C CNN
-F 3 "" H 9350 3950 50  0001 C CNN
-	1    9350 3950
 	1    0    0    -1
 $EndComp
@@
 Wire Wire Line
 	3950 3900 4150 3900
-Text GLabel 8650 4800 2    50   Input ~ 0
+Text GLabel 8650 4750 2    50   Input ~ 0
 IO12
 Text GLabel 10150 4800 2    50   Input ~ 0
@@
 Wire Wire Line
 	10150 4800 10050 4800
-Wire Wire Line
-	8650 4800 8550 4800
-NoConn ~ 8550 5300
 NoConn ~ 10050 5300
 Text GLabel 3950 4400 0    50   Input ~ 0
@@
 Wire Wire Line
 	9050 5300 9050 5450
-Wire Wire Line
-	7700 5300 7550 5300
-Wire Wire Line
-	7550 5300 7550 5350
-Wire Wire Line
-	9500 3850 9350 3850
-Wire Wire Line
-	9350 3850 9350 3950
 Wire Wire Line
 	2100 6000 1900 6000
@@
 F5 "GND" I L 2100 6000 50
 $EndSheet
+$Sheet
+S 7800 4700 500  550
+U 61E0EDBD
+F0 "YL-100" 50
+F1 "pines_sensor2.sch" 50
+F2 "VCC" I L 7800 4800 50
+F3 "Aout" I R 8300 4800 50
+F4 "GND" I L 7800 5100 50
+$EndSheet
+Wire Wire Line
+	8650 4750 8500 4750
+Wire Wire Line
+	8500 4750 8500 4800
+Wire Wire Line
+	8500 4800 8300 4800
+Wire Wire Line
+	7800 4800 7500 4800
+Wire Wire Line
+	7800 5100 7550 5100
+Wire Wire Line
+	7550 5100 7550 5350
 $EndSCHEMATC

Commit message: pcb1
Connections:
- net GND: now also U1.38 (GND)
Changed lines of the file:
@@
 $EndComp
 Wire Wire Line
-	6000 3050 6550 3050
+	6000 3050 6200 3050
 Wire Wire Line
 	6900 3550 6000 3550
@@
 Wire Wire Line
 	7550 5100 7550 5350
+Wire Wire Line
+	6000 3150 6200 3150
+Wire Wire Line
+	6200 3150 6200 3050
+Connection ~ 6200 3050
+Wire Wire Line
+	6200 3050 6550 3050
 $EndSCHEMATC

Commit message: alimentacion
Parts:
- added Cdes1: 100n, Capacitor_SMD:C_0805_2012Metric_Pad1.18x1.45mm_HandSolder, symbol charger_stepup-rescue:C
Connections:
- net +3V3: now also Cdes1.1
- net GND: now also Cdes1.2
Changed lines of the file:
@@
 	2800 2950 2800 2900
 Wire Wire Line
-	3250 2950 2800 2950
-Wire Wire Line
 	3250 3300 3250 2950
 Wire Wire Line
@@
 	2800 2500 2800 2600
 Wire Wire Line
-	3350 2500 2800 2500
+	3350 2500 3150 2500
 Wire Wire Line
 	3350 3200 3350 2500
@@
 Wire Wire Line
 	6200 3050 6550 3050
+$Comp
+L charger_stepup-rescue:C Cdes1
+U 1 1 61E38249
+P 3550 2950
+AR Path="/61E38249" Ref="Cdes1"  Part="1"
+AR Path="/61A8C81F/61E38249" Ref="Cdes"  Part="1"
+F 0 "Cdes1" H 3665 2996 50  0000 L CNN
+F 1 "100n" H 3665 2905 50  0000 L CNN
+F 2 "Capacitor_SMD:C_0805_2012Metric_Pad1.18x1.45mm_HandSolder" H 3588 2800 50  0001 C CNN
+F 3 "" H 3550 2950 50  0001 C CNN
+	1    3550 2950
+	1    0    0    -1
+$EndComp
+Wire Wire Line
+	3550 2800 3150 2500
+Connection ~ 3150 2500
+Wire Wire Line
+	3150 2500 2800 2500
+Wire Wire Line
+	2800 2950 3250 2950
+Wire Wire Line
+	3550 3100 3800 3100
+Connection ~ 3800 3100
 $EndSCHEMATC

Commit message: sensores y cto esp32
Parts:
- SW1, SW2: footprint Button_Switch_SMD:SW_SPST_SKQG_WithStem -> Button_Switch_SMD:SW_SPST_TL3305A
Changed lines of the file:
@@
 F 0 "SW2" H 7050 4717 50  0000 C CNN
 F 1 "SW_DIP_x01" H 7050 4626 50  0000 C CNN
-F 2 "Button_Switch_SMD:SW_SPST_SKQG_WithStem" H 7050 4450 50  0001 C CNN
+F 2 "Button_Switch_SMD:SW_SPST_TL3305A" H 7050 4450 50  0001 C CNN
 F 3 "~" H 7050 4450 50  0001 C CNN
 	1    7050 4450
@@
 F 0 "SW1" H 2800 3617 50  0000 C CNN
 F 1 "SW_DIP_x01" H 2800 3526 50  0000 C CNN
-F 2 "Button_Switch_SMD:SW_SPST_SKQG_WithStem" H 2800 3350 50  0001 C CNN
+F 2 "Button_Switch_SMD:SW_SPST_TL3305A" H 2800 3350 50  0001 C CNN
 F 3 "~" H 2800 3350 50  0001 C CNN
 	1    2800 3350
