File: Diseño PCB/PCB-ESP32S/PCB-ESP32S.sch (KiCad schematic (older format))
At the start: 11 parts, among them J7 Screw_Terminal_01x03, SW1 SW_DIP_x01, SW2 SW_DIP_x01, U1 ESP-32S

Commit message: PCBs ok
Changed lines of the file:
@@
 F6 "ADDR" I R 9150 2700 50
 $EndSheet
-Wire Wire Line
-	8550 2500 8300 2500
-Wire Wire Line
-	8300 2500 8300 2450
 $Comp
 L power:GND #PWR0110
@@
 Wire Wire Line
 	4650 4850 4650 5200
-$Comp
-L power:+3.3V #PWR0109
-U 1 1 61BACFBA
-P 8300 2450
-F 0 "#PWR0109" H 8300 2300 50  0001 C CNN
-F 1 "+3.3V" H 8315 2623 50  0000 C CNN
-F 2 "" H 8300 2450 50  0001 C CNN
-F 3 "" H 8300 2450 50  0001 C CNN
-	1    8300 2450
-	1    0    0    -1
-$EndComp
 $Comp
 L power:+5V #PWR0111
@@
 	3550 3100 3800 3100
 Connection ~ 3800 3100
+$Comp
+L power:+3.3V #PWR0109
+U 1 1 61E330EF
+P 8300 2400
+F 0 "#PWR0109" H 8300 2250 50  0001 C CNN
+F 1 "+3.3V" H 8315 2573 50  0000 C CNN
+F 2 "" H 8300 2400 50  0001 C CNN
+F 3 "" H 8300 2400 50  0001 C CNN
+	1    8300 2400
+	1    0    0    -1
+$EndComp
+Wire Wire Line
+	8550 2500 8300 2500
+Wire Wire Line
+	8300 2500 8300 2400
 $EndSCHEMATC

Commit message: pcv v2
Parts:
- J7: footprint TerminalBlock:TerminalBlock_bornier-3_P5.08mm -> Connector_JST:JST_GH_BM03B-GHS-TBT_1x03-1MP_P1.25mm_Vertical
Changed lines of the file:
@@
 F 0 "J7" H 7330 3192 50  0000 L CNN
 F 1 "Screw_Terminal_01x03" H 7330 3101 50  0000 L CNN
-F 2 "TerminalBlock:TerminalBlock_bornier-3_P5.08mm" H 7250 3150 50  0001 C CNN
+F 2 "Connector_JST:JST_GH_BM03B-GHS-TBT_1x03-1MP_P1.25mm_Vertical" H 7250 3150 50  0001 C CNN
 F 3 "~" H 7250 3150 50  0001 C CNN
 	1    7250 3150

Commit message: mejoras pcb1
Parts:
- SW1: value SW_DIP_x01 -> SW_DIP_x02
- renumbered D9 to D1, D10 to D2, J7 to J1, R16 to R2, R2 to R3, R17 to R4
Changed lines of the file:
@@
 $EndComp
 $Comp
-L Device:R R2
+L Device:R R3
 U 1 1 61A006CD
 P 6550 4150
-F 0 "R2" H 6620 4196 50  0000 L CNN
+F 0 "R3" H 6620 4196 50  0000 L CNN
 F 1 "12K" H 6620 4105 50  0000 L CNN
 F 2 "Resistor_SMD:R_0805_2012Metric_Pad1.20x1.40mm_HandSolder" V 6480 4150 50  0001 C CNN
@@
 P 2800 3350
 F 0 "SW1" H 2800 3617 50  0000 C CNN
-F 1 "SW_DIP_x01" H 2800 3526 50  0000 C CNN
+F 1 "SW_DIP_x02" H 2800 3526 50  0000 C CNN
 F 2 "Button_Switch_SMD:SW_SPST_TL3305A" H 2800 3350 50  0001 C CNN
 F 3 "~" H 2800 3350 50  0001 C CNN
@@
 $EndComp
 $Comp
-L Device:LED D10
+L Device:LED D2
 U 1 1 61BB5D8E
 P 6100 4650
-F 0 "D10" H 6093 4867 50  0000 C CNN
+F 0 "D2" H 6093 4867 50  0000 C CNN
 F 1 "LED" H 6093 4776 50  0000 C CNN
 F 2 "LED_SMD:LED_0805_2012Metric_Pad1.15x1.40mm_HandSolder" H 6100 4650 50  0001 C CNN
@@
 P 7250 3150
 AR Path="/61A61E97/61BBC590" Ref="J?"  Part="1"
-AR Path="/61BBC590" Ref="J7"  Part="1"
-F 0 "J7" H 7330 3192 50  0000 L CNN
+AR Path="/61BBC590" Ref="J1"  Part="1"
+F 0 "J1" H 7330 3192 50  0000 L CNN
 F 1 "Screw_Terminal_01x03" H 7330 3101 50  0000 L CNN
 F 2 "Connector_JST:JST_GH_BM03B-GHS-TBT_1x03-1MP_P1.25mm_Vertical" H 7250 3150 50  0001 C CNN
@@
 	6550 3050 7050 3050
 $Comp
-L Device:R R17
+L Device:R R4
 U 1 1 61BC4B9D
 P 6350 4950
-F 0 "R17" H 6420 4996 50  0000 L CNN
+F 0 "R4" H 6420 4996 50  0000 L CNN
 F 1 "220" H 6420 4905 50  0000 L CNN
 F 2 "Resistor_SMD:R_0805_2012Metric_Pad1.20x1.40mm_HandSolder" V 6280 4950 50  0001 C CNN
@@
 	4750 4950 4750 4850
 $Comp
-L Device:LED D9
+L Device:LED D1
 U 1 1 61BC9643
 P 2250 2750
-F 0 "D9" H 2243 2967 50  0000 C CNN
+F 0 "D1" H 2243 2967 50  0000 C CNN
 F 1 "LED" H 2243 2876 50  0000 C CNN
 F 2 "LED_SMD:LED_0805_2012Metric_Pad1.15x1.40mm_HandSolder" H 2250 2750 50  0001 C CNN
@@
 $EndComp
 $Comp
-L Device:R R16
+L Device:R R2
 U 1 1 61BC9649
 P 2250 3100
-F 0 "R16" H 2320 3146 50  0000 L CNN
+F 0 "R2" H 2320 3146 50  0000 L CNN
 F 1 "220" H 2320 3055 50  0000 L CNN
 F 2 "Resistor_SMD:R_0805_2012Metric_Pad1.20x1.40mm_HandSolder" V 2180 3100 50  0001 C CNN

Commit message: edicion true hole
Parts:
- J1: footprint Connector_JST:JST_GH_BM03B-GHS-TBT_1x03-1MP_P1.25mm_Vertical -> Connector_JST:JST_EH_B3B-EH-A_1x03_P2.50mm_Vertical
Changed lines of the file:
@@
 F 0 "J1" H 7330 3192 50  0000 L CNN
 F 1 "Screw_Terminal_01x03" H 7330 3101 50  0000 L CNN
-F 2 "Connector_JST:JST_GH_BM03B-GHS-TBT_1x03-1MP_P1.25mm_Vertical" H 7250 3150 50  0001 C CNN
+F 2 "Connector_JST:JST_EH_B3B-EH-A_1x03_P2.50mm_Vertical" H 7250 3150 50  0001 C CNN
 F 3 "~" H 7250 3150 50  0001 C CNN
 	1    7250 3150
