File: Diseño PCB/PCB-ESP32S/alimentacion.sch (KiCad schematic (older format))
At the start: 12 parts

Commit message: esp-32 actualizacion
Parts:
- D8: renamed from D?; footprint (none) -> LED_SMD:LED_0805_2012Metric_Pad1.15x1.40mm_HandSolder
- R13, R14, R15: renamed from R?; footprint (none) -> Resistor_SMD:R_0805_2012Metric_Pad1.20x1.40mm_HandSolder
- U6: renamed from U?; footprint (none) -> Package_TO_SOT_THT:TO-220-3_Vertical
- gave numbers to parts that had none: 7
Changed lines of the file:
@@
 $Descr A4 11693 8268
 encoding utf-8
-Sheet 7 8
+Sheet 6 8
 Title ""
 Date ""
@@
 $EndDescr
 $Comp
-L pspice:CAP C?
+L pspice:CAP C5
 U 1 1 61A64F42
 P 3600 3250
-F 0 "C?" H 3778 3296 50  0000 L CNN
+F 0 "C5" H 3778 3296 50  0000 L CNN
 F 1 "100u" H 3778 3205 50  0000 L CNN
 F 2 "" H 3600 3250 50  0001 C CNN
@@
 $EndComp
 $Comp
-L pspice:CAP C?
+L pspice:CAP C7
 U 1 1 61A6675D
 P 4700 3250
-F 0 "C?" H 4878 3296 50  0000 L CNN
+F 0 "C7" H 4878 3296 50  0000 L CNN
 F 1 "100u" H 4878 3205 50  0000 L CNN
 F 2 "" H 4700 3250 50  0001 C CNN
@@
 	4700 3500 4700 3850
 $Comp
-L Device:LED D?
+L Device:LED D7
 U 1 1 61A6F4A6
 P 5250 3600
-F 0 "D?" H 5243 3817 50  0000 C CNN
+F 0 "D7" H 5243 3817 50  0000 C CNN
 F 1 "LED" H 5243 3726 50  0000 C CNN
 F 2 "" H 5250 3600 50  0001 C CNN
@@
 $EndComp
 $Comp
-L Device:R R?
+L Device:R R14
 U 1 1 61A71AC0
 P 5250 3250
-F 0 "R?" H 5320 3296 50  0000 L CNN
+F 0 "R14" H 5320 3296 50  0000 L CNN
 F 1 "680" H 5320 3205 50  0000 L CNN
-F 2 "" V 5180 3250 50  0001 C CNN
+F 2 "Resistor_SMD:R_0805_2012Metric_Pad1.20x1.40mm_HandSolder" V 5180 3250 50  0001 C CNN
 F 3 "~" H 5250 3250 50  0001 C CNN
 	1    5250 3250
@@
 	5250 3450 5250 3400
 $Comp
-L Regulator_Linear:LM7805_TO220 U?
+L Regulator_Linear:LM7805_TO220 U5
 U 1 1 61A72BA8
 P 4200 2900
-F 0 "U?" H 4200 3142 50  0000 C CNN
+F 0 "U5" H 4200 3142 50  0000 C CNN
 F 1 "LM7805_TO220" H 4200 3051 50  0000 C CNN
 F 2 "Package_TO_SOT_THT:TO-220-3_Vertical" H 4200 3125 50  0001 C CIN
@@
 	5250 2950 5750 2950
 $Comp
-L pspice:CAP C?
+L pspice:CAP C6
 U 1 1 61A8758A
 P 3600 4800
-F 0 "C?" H 3778 4846 50  0000 L CNN
+F 0 "C6" H 3778 4846 50  0000 L CNN
 F 1 "10u" H 3778 4755 50  0000 L CNN
 F 2 "" H 3600 4800 50  0001 C CNN
@@
 $EndComp
 $Comp
-L pspice:CAP C?
+L pspice:CAP C8
 U 1 1 61A87590
 P 4700 4800
-F 0 "C?" H 4878 4846 50  0000 L CNN
+F 0 "C8" H 4878 4846 50  0000 L CNN
 F 1 "10u" H 4878 4755 50  0000 L CNN
 F 2 "" H 4700 4800 50  0001 C CNN
@@
 	4700 5050 4700 5400
 $Comp
-L Device:LED D?
+L Device:LED D8
 U 1 1 61A875AB
 P 5250 5150
-F 0 "D?" H 5243 5367 50  0000 C CNN
+F 0 "D8" H 5243 5367 50  0000 C CNN
 F 1 "LED" H 5243 5276 50  0000 C CNN
-F 2 "" H 5250 5150 50  0001 C CNN
+F 2 "LED_SMD:LED_0805_2012Metric_Pad1.15x1.40mm_HandSolder" H 5250 5150 50  0001 C CNN
 F 3 "~" H 5250 5150 50  0001 C CNN
 	1    5250 5150
@@
 $EndComp
 $Comp
-L Device:R R?
+L Device:R R15
 U 1 1 61A875B1
 P 5250 4800
-F 0 "R?" H 5320 4846 50  0000 L CNN
+F 0 "R15" H 5320 4846 50  0000 L CNN
 F 1 "470" H 5320 4755 50  0000 L CNN
-F 2 "" V 5180 4800 50  0001 C CNN
+F 2 "Resistor_SMD:R_0805_2012Metric_Pad1.20x1.40mm_HandSolder" V 5180 4800 50  0001 C CNN
 F 3 "~" H 5250 4800 50  0001 C CNN
 	1    5250 4800
@@
 Connection ~ 5250 4450
 $Comp
-L Regulator_Linear:LM1117-3.3 U?
+L Regulator_Linear:LM1117-3.3 U6
 U 1 1 61A88682
 P 4200 4450
-F 0 "U?" H 4200 4692 50  0000 C CNN
+F 0 "U6" H 4200 4692 50  0000 C CNN
 F 1 "LM1117-3.3" H 4200 4601 50  0000 C CNN
-F 2 "" H 4200 4450 50  0001 C CNN
+F 2 "Package_TO_SOT_THT:TO-220-3_Vertical" H 4200 4450 50  0001 C CNN
 F 3 "http://www.ti.com/lit/ds/symlink/lm1117.pdf" H 4200 4450 50  0001 C CNN
 	1    4200 4450
@@
 $EndComp
 $Comp
-L Device:R R?
+L Device:R R13
 U 1 1 61A8B0C5
 P 3350 2900
-F 0 "R?" H 3420 2946 50  0000 L CNN
+F 0 "R13" H 3420 2946 50  0000 L CNN
 F 1 "2" H 3420 2855 50  0000 L CNN
-F 2 "" V 3280 2900 50  0001 C CNN
+F 2 "Resistor_SMD:R_0805_2012Metric_Pad1.20x1.40mm_HandSolder" V 3280 2900 50  0001 C CNN
 F 3 "~" H 3350 2900 50  0001 C CNN
 	1    3350 2900
@@
 $EndComp
 $Comp
-L Transistor_BJT:TIP42C Q?
+L Transistor_BJT:TIP42C Q3
 U 1 1 61A8E37D
 P 3600 2500
-F 0 "Q?" H 3791 2546 50  0000 L CNN
+F 0 "Q3" H 3791 2546 50  0000 L CNN
 F 1 "TIP42C" H 3791 2455 50  0000 L CNN
 F 2 "Package_TO_SOT_THT:TO-220-3_Vertical" H 3850 2425 50  0001 L CIN

Commit message: Actualización
Parts:
- added J?: Screw_Terminal_01x02, TerminalBlock:TerminalBlock_bornier-2_P5.08mm, symbol Connector:Screw_Terminal_01x02
- C5, C7: footprint (none) -> Capacitor_SMD:C_Elec_4x5.8
- C6, C8: footprint (none) -> Capacitor_SMD:C_1206_3216Metric_Pad1.33x1.80mm_HandSolder
- D7: footprint (none) -> LED_SMD:LED_0805_2012Metric_Pad1.15x1.40mm_HandSolder
Connections:
- net GND: now also J?.2 (Pin_2)
- net 12V renamed 12v
- net 12v: now also J?.1 (Pin_1)
Changed lines of the file:
@@
 $Descr A4 11693 8268
 encoding utf-8
-Sheet 6 8
+Sheet 6 7
 Title ""
 Date ""
@@
 F 0 "C5" H 3778 3296 50  0000 L CNN
 F 1 "100u" H 3778 3205 50  0000 L CNN
-F 2 "" H 3600 3250 50  0001 C CNN
+F 2 "Capacitor_SMD:C_Elec_4x5.8" H 3600 3250 50  0001 C CNN
 F 3 "~" H 3600 3250 50  0001 C CNN
 	1    3600 3250
@@
 F 0 "C7" H 4878 3296 50  0000 L CNN
 F 1 "100u" H 4878 3205 50  0000 L CNN
-F 2 "" H 4700 3250 50  0001 C CNN
+F 2 "Capacitor_SMD:C_Elec_4x5.8" H 4700 3250 50  0001 C CNN
 F 3 "~" H 4700 3250 50  0001 C CNN
 	1    4700 3250
@@
 F 0 "D7" H 5243 3817 50  0000 C CNN
 F 1 "LED" H 5243 3726 50  0000 C CNN
-F 2 "" H 5250 3600 50  0001 C CNN
+F 2 "LED_SMD:LED_0805_2012Metric_Pad1.15x1.40mm_HandSolder" H 5250 3600 50  0001 C CNN
 F 3 "~" H 5250 3600 50  0001 C CNN
 	1    5250 3600
@@
 F 0 "C6" H 3778 4846 50  0000 L CNN
 F 1 "10u" H 3778 4755 50  0000 L CNN
-F 2 "" H 3600 4800 50  0001 C CNN
+F 2 "Capacitor_SMD:C_1206_3216Metric_Pad1.33x1.80mm_HandSolder" H 3600 4800 50  0001 C CNN
 F 3 "~" H 3600 4800 50  0001 C CNN
 	1    3600 4800
@@
 F 0 "C8" H 4878 4846 50  0000 L CNN
 F 1 "10u" H 4878 4755 50  0000 L CNN
-F 2 "" H 4700 4800 50  0001 C CNN
+F 2 "Capacitor_SMD:C_1206_3216Metric_Pad1.33x1.80mm_HandSolder" H 4700 4800 50  0001 C CNN
 F 3 "~" H 4700 4800 50  0001 C CNN
 	1    4700 4800
@@
 Connection ~ 5250 5400
 Wire Wire Line
-	3000 3850 3000 5400
+	3000 3850 3000 4350
 Wire Wire Line
 	3000 3850 3600 3850
@@
 Text HLabel 5750 2950 3    50   Input ~ 0
 5V
-Text HLabel 2900 2900 3    50   Input ~ 0
-12V
 Text HLabel 5750 4450 3    50   Input ~ 0
 3.3V
@@
 Wire Wire Line
 	5250 2950 5250 3100
+$Comp
+L Connector:Screw_Terminal_01x02 J?
+U 1 1 61BB9845
+P 2350 4250
+F 0 "J?" H 2268 4467 50  0000 C CNN
+F 1 "Screw_Terminal_01x02" H 2268 4376 50  0000 C CNN
+F 2 "TerminalBlock:TerminalBlock_bornier-2_P5.08mm" H 2350 4250 50  0001 C CNN
+F 3 "~" H 2350 4250 50  0001 C CNN
+	1    2350 4250
+	-1   0    0    -1
+$EndComp
+Wire Wire Line
+	2550 4250 2900 4250
+Wire Wire Line
+	2900 4250 2900 2900
+Wire Wire Line
+	2550 4350 3000 4350
+Connection ~ 3000 4350
+Wire Wire Line
+	3000 4350 3000 5400
+Text HLabel 2900 2900 0    50   Input ~ 0
+12v
 $EndSCHEMATC

Commit message: Actualización2
Parts:
- C5, C7: footprint Capacitor_SMD:C_Elec_4x5.8 -> Capacitor_SMD:CP_Elec_6.3x5.8
Changed lines of the file:
@@
 $Descr A4 11693 8268
 encoding utf-8
-Sheet 6 7
+Sheet 5 7
 Title ""
 Date ""
@@
 F 0 "C5" H 3778 3296 50  0000 L CNN
 F 1 "100u" H 3778 3205 50  0000 L CNN
-F 2 "Capacitor_SMD:C_Elec_4x5.8" H 3600 3250 50  0001 C CNN
+F 2 "Capacitor_SMD:CP_Elec_6.3x5.8" H 3600 3250 50  0001 C CNN
 F 3 "~" H 3600 3250 50  0001 C CNN
 	1    3600 3250
@@
 F 0 "C7" H 4878 3296 50  0000 L CNN
 F 1 "100u" H 4878 3205 50  0000 L CNN
-F 2 "Capacitor_SMD:C_Elec_4x5.8" H 4700 3250 50  0001 C CNN
+F 2 "Capacitor_SMD:CP_Elec_6.3x5.8" H 4700 3250 50  0001 C CNN
 F 3 "~" H 4700 3250 50  0001 C CNN
 	1    4700 3250
