File: Diseño PCB/PCB-ESP32S/_autosave-PCB-ESP32S.kicad_pcb (KiCad board)
At the start: 2 copper layers, 39 parts, among them J1 Screw_Terminal_01x03, J3 Screw_Terminal_01x03, J7 Screw_Terminal_01x03, J8 Screw_Terminal_01x02, K1 SRD-05VDC-SL-C, K2 SRD-05VDC-SL-C, Q1 MMBT2222A, Q2 MMBT2222A, Q3 TIP42C, SW1 SW_DIP_x01, SW2 SW_DIP_x01, U1 ESP-32S, U3 PC817, U4 PC817, U5 LM7805_TO220, U6 LM1117-3.3

Commit message: reles
Parts:
- removed D1, D3: LED, LED_SMD:LED_0805_2012Metric_Pad1.15x1.40mm_HandSolder
- removed D2, D4: 1N4007, Diode_SMD:D_SMA_Handsoldering
- removed J1, J3: Screw_Terminal_01x03, TerminalBlock:TerminalBlock_bornier-3_P5.08mm
- removed K1, K2: SRD-05VDC-SL-C, ModuloRele:RELAY_SRD-05VDC-SL-C
- removed Q1, Q2: MMBT2222A, ModuloRele:SOT23
- removed R11, R4, R5, R6: R, Resistor_SMD:R_0805_2012Metric_Pad1.20x1.40mm_HandSolder
- removed U3, U4: PC817, Package_DIP:DIP-4_W7.62mm
- added C1: 0.1uF, Capacitor_SMD:C_0805_2012Metric_Pad1.18x1.45mm_HandSolder, F.Cu at (246.4, 148.6)
- added IC1: BH1750FVI-TR, BH1750:WSOF6, F.Cu at (243.8, 156.2)
- added R10: 4.7k, Resistor_SMD:R_0805_2012Metric_Pad1.20x1.40mm_HandSolder, F.Cu at (235.9, 142.5)
- added R3: 1k, Resistor_SMD:R_0805_2012Metric_Pad1.20x1.40mm_HandSolder, F.Cu at (182.9, 162.6)
- added R7: 1k, Resistor_SMD:R_0805_2012Metric_Pad1.20x1.40mm_HandSolder, F.Cu at (235.9, 139.5)
- added R8: 4.7k, Resistor_SMD:R_0805_2012Metric_Pad1.20x1.40mm_HandSolder, F.Cu at (240.6, 142.5)
- added R9: 4.7k, Resistor_SMD:R_0805_2012Metric_Pad1.20x1.40mm_HandSolder, F.Cu at (237.5, 149.9)
- added TH1: DHT22_Temperature_Humidity, Sensors:DHT22_Temperature_Humidity, F.Cu at (185.4, 148.6)
- added u2: Conn_01x04_Male, Connector_JST:JST_GH_BM04B-GHS-TBT_1x04-1MP_P1.25mm_Vertical, F.Cu at (247.3, 46.5)
- added u7: Conn_01x04_Male, Connector_JST:JST_GH_BM04B-GHS-TBT_1x04-1MP_P1.25mm_Vertical, F.Cu at (246.4, 54.6)
- U5: moved to B.Cu
- moved C6 144.9 mm to (139.7, 110.5)
- moved C7 142.7 mm to (124.5, 104.1)
- moved C8 129.0 mm to (130.8, 110.5)
- moved D7 127.1 mm to (134.6, 104.1)
- moved R17 90.1 mm to (214.6, 127.0)
- moved C5 83.0 mm to (193.0, 91.4), turned to 270 degrees
- moved J7 80.7 mm to (241.3, 102.9), turned to 270 degrees
- moved D9 80.1 mm to (206.7, 122.1)
- moved D10 80.1 mm to (201.9, 122.1)
- moved J8 78.2 mm to (177.8, 82.5), turned to 90 degrees
- moved U1 76.6 mm to (224.8, 87.6)
- moved R16 69.5 mm to (226.1, 105.4)
- moved U6 65.6 mm to (193.0, 102.9)
- moved U5 49.7 mm to (198.1, 81.3)
- moved SW2 48.1 mm to (229.9, 115.6)
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Connections:
- U1 pad 13: (no net) -> IO14
- U1 pad 14: (no net) -> IO12
- U1 pad 24: (no net) -> IO2
- U1 pad 8: (no net) -> IO32
- U1 pad 9: (no net) -> IO33
Routing:
- net GND: track 0.00 -> 47.4 mm
- net Net-(J7-Pad3): track 0.00 -> 35.5 mm
- net Net-(J7-Pad2): track 0.00 -> 31.7 mm
