File: Diseño PCB/PCB-ESP32S/PCB-ESP32S.kicad_pcb (KiCad board)
At the start: 2 copper layers, 2 parts, among them U1 ESP-32S

Commit message: actualizando dibujo
Parts:
- removed REF**: DHT22_Temperature_Humidity, Sensors:DHT22_Temperature_Humidity
- added R1: 12K, Resistor_SMD:R_0603_1608Metric, F.Cu at (172.7, 102.9)
- added R2: 12K, Resistor_SMD:R_0603_1608Metric, F.Cu at (176.7, 102.9)
- added SW1: SW_DIP_x01, Button_Switch_SMD:SW_SPST_SKQG_WithStem, F.Cu at (175.5, 98.2)
- added SW2: SW_DIP_x01, Button_Switch_SMD:SW_SPST_SKQG_WithStem, F.Cu at (185.0, 98.2)
Connections:
- U1 pad 1: (no net) -> GND
- U1 pad 15: (no net) -> GND
- U1 pad 2: (no net) -> +3V3
- U1 pad 25: (no net) -> Net-(R2-Pad2)
- U1 pad 3: (no net) -> Net-(R1-Pad2)
- U1 pad 39: (no net) -> GND

Commit message: esp-32 actualizacion
Parts:
- added D1: LED, LED_SMD:LED_0805_2012Metric_Pad1.15x1.40mm_HandSolder, F.Cu at (135.9, 50.8)
- added D2: 1N4007, Diode_SMD:D_SMA_Handsoldering, F.Cu at (149.3, 38.2)
- added D3: LED, LED_SMD:LED_0805_2012Metric_Pad1.15x1.40mm_HandSolder, F.Cu at (129.3, 55.5)
- added D4: 1N4007, Diode_SMD:D_SMA_Handsoldering, F.Cu at (121.8, 56.3)
- added D5: VS-KBPC104, Diode_THT:Diode_Bridge_Vishay_KBPC1, F.Cu at (139.8, 65.2)
- added D6: 1N5349B, Diode_THT:D_DO-201_P15.24mm_Horizontal, F.Cu at (118.9, 64.9)
- added D8: LED, LED_SMD:LED_0805_2012Metric_Pad1.15x1.40mm_HandSolder, F.Cu at (174.1, 43.4)
- added IC1: BH1750FVI-TR, BH1750:WSOF6, F.Cu at (169.2, 78.5)
- added J1: Screw_Terminal_01x03, TerminalBlock:TerminalBlock_bornier-3_P5.08mm, F.Cu at (120.1, 49.5)
- added J3: Screw_Terminal_01x03, TerminalBlock:TerminalBlock_bornier-3_P5.08mm, F.Cu at (120.1, 40.4)
- added J7: Screw_Terminal_01x03, TerminalBlock:TerminalBlock_bornier-3_P5.08mm, F.Cu at (190.1, 40.4)
- added Q3: TIP42C, Package_TO_SOT_THT:TO-220-3_Vertical, F.Cu at (163.3, 39.8)
- added R10: 4.7k, Resistor_SMD:R_0805_2012Metric_Pad1.20x1.40mm_HandSolder, F.Cu at (159.7, 81.5)
- added R11: R, Resistor_SMD:R_0805_2012Metric_Pad1.20x1.40mm_HandSolder, F.Cu at (146.7, 41.9)
- added R13: 2, Resistor_SMD:R_0805_2012Metric_Pad1.20x1.40mm_HandSolder, F.Cu at (178.8, 43.3)
- added R14: 680, Resistor_SMD:R_0805_2012Metric_Pad1.20x1.40mm_HandSolder, F.Cu at (174.0, 46.4)
- added R15: 470, Resistor_SMD:R_0805_2012Metric_Pad1.20x1.40mm_HandSolder, F.Cu at (178.8, 46.3)
- added R16: 220, Resistor_SMD:R_0805_2012Metric_Pad1.20x1.40mm_HandSolder, F.Cu at (189.3, 46.4)
- added R17: 220, Resistor_SMD:R_0805_2012Metric_Pad1.20x1.40mm_HandSolder, F.Cu at (205.9, 37.4)
- added R3: 1k, Resistor_SMD:R_0805_2012Metric_Pad1.20x1.40mm_HandSolder, F.Cu at (159.7, 71.8)
- added R4: R, Resistor_SMD:R_0805_2012Metric_Pad1.20x1.40mm_HandSolder, F.Cu at (146.7, 44.9)
- added R5: R, Resistor_SMD:R_0805_2012Metric_Pad1.20x1.40mm_HandSolder, F.Cu at (151.4, 41.9)
- added R6: R, Resistor_SMD:R_0805_2012Metric_Pad1.20x1.40mm_HandSolder, F.Cu at (134.0, 55.5)
- added R7: 1k, Resistor_SMD:R_0805_2012Metric_Pad1.20x1.40mm_HandSolder, F.Cu at (159.7, 78.6)
- added R8: 4.7k, Resistor_SMD:R_0805_2012Metric_Pad1.20x1.40mm_HandSolder, F.Cu at (164.4, 81.5)
- added R9: 4.7k, Resistor_SMD:R_0805_2012Metric_Pad1.20x1.40mm_HandSolder, F.Cu at (164.4, 78.6)
- added TH1: DHT22_Temperature_Humidity, Sensors:DHT22_Temperature_Humidity, F.Cu at (165.5, 65.4)
- added U2: pines_sensor, Connector_JST:JST_GH_SM04B-GHS-TB_1x04-1MP_P1.25mm_Horizontal, F.Cu at (187.8, 56.0)
- added U3: PC817, Package_DIP:DIP-4_W7.62mm, F.Cu at (135.1, 38.0)
- added U4: PC817, Package_DIP:DIP-4_W7.62mm, F.Cu at (135.1, 44.7)
- added U5: LM7805_TO220, Package_TO_SOT_THT:TO-220-3_Vertical, F.Cu at (163.3, 45.8)
- added U6: LM1117-3.3, Package_TO_SOT_THT:TO-220-3_Vertical, F.Cu at (174.9, 39.8)
- added U7: pines_sensor, Connector_JST:JST_GH_SM04B-GHS-TB_1x04-1MP_P1.25mm_Horizontal, F.Cu at (187.8, 67.0)
- R1, R2: footprint Resistor_SMD:R_0603_1608Metric -> Resistor_SMD:R_0805_2012Metric_Pad1.20x1.40mm_HandSolder
Connections:
- U1 pad 26: (no net) -> IO4
- U1 pad 34: (no net) -> Net-(J7-Pad3)
- U1 pad 35: (no net) -> Net-(J7-Pad2)

Commit message: verificacion componentes
Parts:
- removed D5: VS-KBPC104, Diode_THT:Diode_Bridge_Vishay_KBPC1
- removed D6: 1N5349B, Diode_THT:D_DO-201_P15.24mm_Horizontal
- added C1: 0.1uF, Capacitor_SMD:C_0805_2012Metric_Pad1.18x1.45mm_HandSolder, F.Cu at (242.9, 59.5)
- added C1b1: 0.1uF, Capacitor_SMD:C_0805_2012Metric_Pad1.18x1.45mm_HandSolder, F.Cu at (213.0, 68.8)
- added C2b1: 10uF, Capacitor_SMD:C_0805_2012Metric_Pad1.18x1.45mm_HandSolder, F.Cu at (204.5, 75.3)
- added C3b1: 0.1uF, Capacitor_SMD:C_0805_2012Metric_Pad1.18x1.45mm_HandSolder, F.Cu at (209.3, 75.3)
- added C5: 100u, Capacitor_SMD:CP_Elec_6.3x5.8, F.Cu at (253.1, 34.1)
- added C6: 10u, Capacitor_SMD:C_1206_3216Metric_Pad1.33x1.80mm_HandSolder, F.Cu at (261.3, 31.7)
- added C7: 100u, Capacitor_SMD:CP_Elec_6.3x5.8, F.Cu at (253.1, 42.2)
- added C8: 10u, Capacitor_SMD:C_1206_3216Metric_Pad1.33x1.80mm_HandSolder, F.Cu at (239.3, 40.7)
- added D10: LED, LED_SMD:LED_0805_2012Metric_Pad1.15x1.40mm_HandSolder, F.Cu at (238.7, 51.0)
- added D1b1: LED, LED_SMD:LED_0805_2012Metric_Pad1.15x1.40mm_HandSolder, F.Cu at (218.0, 68.8)
- added D2b1: LED, LED_SMD:LED_0805_2012Metric_Pad1.15x1.40mm_HandSolder, F.Cu at (213.0, 71.9)
- added D7: LED, LED_SMD:LED_0805_2012Metric_Pad1.15x1.40mm_HandSolder, F.Cu at (244.7, 40.6)
- added D9: LED, LED_SMD:LED_0805_2012Metric_Pad1.15x1.40mm_HandSolder, F.Cu at (243.5, 51.0)
- added J10: CONN_in+, Connector_PinHeader_2.54mm:PinHeader_1x01_P2.54mm_Horizontal, F.Cu at (191.1, 69.7)
- added J11: CONN_in-, Connector_PinHeader_2.54mm:PinHeader_1x01_P2.54mm_Horizontal, F.Cu at (204.5, 60.4)
- added J2: Screw_Terminal_01x05, Connector_JST:JST_GH_BM05B-GHS-TBT_1x05-1MP_P1.25mm_Vertical, F.Cu at (234.6, 61.9)
- added J4: CONN_bat+, Connector_PinHeader_2.54mm:PinHeader_1x01_P2.54mm_Horizontal, F.Cu at (191.1, 60.4)
- added J5: CONN_bat-, Connector_PinHeader_2.54mm:PinHeader_1x01_P2.54mm_Horizontal, F.Cu at (191.1, 65.0)
- added J6: CONN_out-, Connector_PinHeader_2.54mm:PinHeader_1x01_P2.54mm_Horizontal, F.Cu at (191.1, 74.3)
- added J8: Screw_Terminal_01x02, TerminalBlock:TerminalBlock_bornier-2_P5.08mm, F.Cu at (239.5, 34.5)
- added J9: CONN_out+, Connector_PinHeader_2.54mm:PinHeader_1x01_P2.54mm_Horizontal, F.Cu at (204.5, 65.0)
- added K1: SRD-05VDC-SL-C, ModuloRele:RELAY_SRD-05VDC-SL-C, F.Cu at (199.7, 38.5)
- added K2: SRD-05VDC-SL-C, ModuloRele:RELAY_SRD-05VDC-SL-C, F.Cu at (221.0, 38.5)
- added Q1: MMBT2222A, ModuloRele:SOT23, F.Cu at (190.7, 49.3)
- added Q2: MMBT2222A, ModuloRele:SOT23, F.Cu at (194.7, 49.3)
- added R1b1: 1k, Resistor_SMD:R_0805_2012Metric_Pad1.20x1.40mm_HandSolder, F.Cu at (214.1, 74.9)
- added R2b1: 1k, Resistor_SMD:R_0805_2012Metric_Pad1.20x1.40mm_HandSolder, F.Cu at (217.7, 71.8)
- added R4b1: 1k, Resistor_SMD:R_0805_2012Metric_Pad1.20x1.40mm_HandSolder, F.Cu at (222.7, 68.7)
- added R5b1: 100, Resistor_SMD:R_0805_2012Metric_Pad1.20x1.40mm_HandSolder, F.Cu at (218.9, 74.8)
- added Rprog1: 10k, Resistor_SMD:R_0805_2012Metric_Pad1.20x1.40mm_HandSolder, F.Cu at (222.5, 71.7)
- added U1b1: TP4056, lib:TP4056_SOP-8-PP, F.Cu at (206.4, 70.6)
- added U2b1: DW01, Package_TO_SOT_SMD:SOT-23-6_Handsoldering, F.Cu at (218.5, 64.9)
- added U3b1: FS8205A, Package_SO:TSSOP-8_4.4x3mm_P0.65mm, F.Cu at (219.9, 60.3)
Connections:
- net /Sheet61A8C81E/12V renamed /Sheet61A8C81E/12v
- D2 pad 2: (no net) -> Net-(D2-Pad2)
- D4 pad 2: (no net) -> Net-(D4-Pad2)
- IC1 pad 1: +5V -> +3V3
- R10 pad 1: +5V -> +3V3
- R11 pad 2: (no net) -> Net-(Q2-Pad1)
- R14 pad 2: (no net) -> Net-(D7-Pad2)
- R16 pad 1: (no net) -> Net-(D9-Pad2)
- R17 pad 1: (no net) -> Net-(D10-Pad2)
- R6 pad 2: (no net) -> Net-(Q1-Pad1)
- R7 pad 2: +5V -> +3V3
- R9 pad 1: +5V -> +3V3
- U1 pad 16: (no net) -> Net-(D10-Pad1)

Commit message: separacion
Parts:
- removed C1b1, C3b1: 0.1uF, Capacitor_SMD:C_0805_2012Metric_Pad1.18x1.45mm_HandSolder
- removed C2b1: 10uF, Capacitor_SMD:C_0805_2012Metric_Pad1.18x1.45mm_HandSolder
- removed D1, D1b1, D2b1, D3: LED, LED_SMD:LED_0805_2012Metric_Pad1.15x1.40mm_HandSolder
- removed D2, D4: 1N4007, Diode_SMD:D_SMA_Handsoldering
- removed J1, J3: Screw_Terminal_01x03, TerminalBlock:TerminalBlock_bornier-3_P5.08mm
- removed J10: CONN_in+, Connector_PinHeader_2.54mm:PinHeader_1x01_P2.54mm_Horizontal
- removed J11: CONN_in-, Connector_PinHeader_2.54mm:PinHeader_1x01_P2.54mm_Horizontal
- removed J2: Screw_Terminal_01x05, Connector_JST:JST_GH_BM05B-GHS-TBT_1x05-1MP_P1.25mm_Vertical
- removed J4: CONN_bat+, Connector_PinHeader_2.54mm:PinHeader_1x01_P2.54mm_Horizontal
- removed J5: CONN_bat-, Connector_PinHeader_2.54mm:PinHeader_1x01_P2.54mm_Horizontal
- removed J6: CONN_out-, Connector_PinHeader_2.54mm:PinHeader_1x01_P2.54mm_Horizontal
- removed J9: CONN_out+, Connector_PinHeader_2.54mm:PinHeader_1x01_P2.54mm_Horizontal
- removed K1, K2: SRD-05VDC-SL-C, ModuloRele:RELAY_SRD-05VDC-SL-C
- removed Q1, Q2: MMBT2222A, ModuloRele:SOT23
- removed R11, R4, R5, R6: R, Resistor_SMD:R_0805_2012Metric_Pad1.20x1.40mm_HandSolder
- removed R1b1, R2b1, R4b1: 1k, Resistor_SMD:R_0805_2012Metric_Pad1.20x1.40mm_HandSolder
- removed R5b1: 100, Resistor_SMD:R_0805_2012Metric_Pad1.20x1.40mm_HandSolder
- removed Rprog1: 10k, Resistor_SMD:R_0805_2012Metric_Pad1.20x1.40mm_HandSolder
- removed U1b1: TP4056, lib:TP4056_SOP-8-PP
- removed U2, U7: pines_sensor, Connector_JST:JST_GH_SM04B-GHS-TB_1x04-1MP_P1.25mm_Horizontal
- removed U2b1: DW01, Package_TO_SOT_SMD:SOT-23-6_Handsoldering
- removed U3, U4: PC817, Package_DIP:DIP-4_W7.62mm
- removed U3b1: FS8205A, Package_SO:TSSOP-8_4.4x3mm_P0.65mm
- added u2: Conn_01x04_Male, Connector_JST:JST_GH_BM04B-GHS-TBT_1x04-1MP_P1.25mm_Vertical, F.Cu at (247.3, 46.5)
- added u7: Conn_01x04_Male, Connector_JST:JST_GH_BM04B-GHS-TBT_1x04-1MP_P1.25mm_Vertical, F.Cu at (246.4, 54.6)
- moved C6 144.9 mm to (139.7, 110.5)
- moved C7 142.7 mm to (124.5, 104.1)
- moved C5 133.3 mm to (134.6, 95.2)
- moved C8 129.0 mm to (130.8, 110.5)
- moved D7 127.1 mm to (134.6, 104.1)
- moved IC1 107.7 mm to (243.8, 156.2)
- moved R9 102.1 mm to (237.5, 149.9)
- moved R10 97.6 mm to (235.9, 142.5)
- moved R8 97.6 mm to (240.6, 142.5)
- moved R7 97.6 mm to (235.9, 139.5)
- moved R3 93.7 mm to (182.9, 162.6)
- moved R17 90.1 mm to (214.6, 127.0)
- moved C1 89.1 mm to (246.4, 148.6)
- moved TH1 85.5 mm to (185.4, 148.6)
- moved J7 80.7 mm to (241.3, 102.9), turned to 270 degrees
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Connections:
- C5 pad 2: /Sheet61A8C81E/GND -> GND
- C6 pad 2: /Sheet61A8C81E/GND -> GND
- C7 pad 1: /Sheet61A8C81E/5V -> +5V
- C7 pad 2: /Sheet61A8C81E/GND -> GND
- C8 pad 1: /Sheet61A8C81E/3.3V -> +3V3
- C8 pad 2: /Sheet61A8C81E/GND -> GND
- D7 pad 1: /Sheet61A8C81E/GND -> GND
- D8 pad 1: /Sheet61A8C81E/GND -> GND
- IC1 pad 4: /BH1750/SDA -> IO33
- IC1 pad 6: /BH1750/SCL -> IO32
- J8 pad 2: /Sheet61A8C81E/GND -> GND
- Q3 pad 2: /Sheet61A8C81E/5V -> +5V
- R10 pad 2: /BH1750/SCL -> IO33
- R14 pad 1: /Sheet61A8C81E/5V -> +5V
- R15 pad 1: /Sheet61A8C81E/3.3V -> +3V3
- R3 pad 2: IO4 -> IO2
- R9 pad 2: /BH1750/SDA -> IO32
- TH1 pad 2: IO4 -> IO2
- U1 pad 13: (no net) -> IO14
- U1 pad 14: (no net) -> IO12
- U1 pad 24: (no net) -> IO2
- U1 pad 26: IO4 -> (no net)
- U1 pad 8: (no net) -> IO32
- U1 pad 9: (no net) -> IO33
- U5 pad 2: /Sheet61A8C81E/GND -> GND
- U5 pad 3: /Sheet61A8C81E/5V -> +5V
- U6 pad 1: /Sheet61A8C81E/GND -> GND
- U6 pad 2: /Sheet61A8C81E/3.3V -> +3V3
Routing:
- net GND: track 0.00 -> 47.4 mm
- net Net-(J7-Pad3): track 0.00 -> 35.5 mm
- net Net-(J7-Pad2): track 0.00 -> 31.7 mm

Commit message: pcb1
Parts:
- moved C7 78.5 mm to (196.8, 73.7), turned to 90 degrees
- moved D7 77.8 mm to (205.1, 71.1), turned to 270 degrees
- moved C8 75.0 mm to (200.7, 83.2), turned to 90 degrees
- moved D8 54.9 mm to (207.0, 83.2), turned to 270 degrees
- moved C6 54.8 mm to (188.6, 85.7), turned to 270 degrees
- moved R14 53.0 mm to (205.1, 76.2), turned to 90 degrees
- moved R15 49.5 mm to (206.7, 88.3), turned to 90 degrees
- moved U6 48.3 mm to (194.9, 88.3), turned to 90 degrees
- moved Q3 44.0 mm to (177.8, 81.9)
- moved U5 39.2 mm to (171.4, 73.7)
- moved R13 33.0 mm to (171.4, 85.1), turned to 90 degrees
- moved C5 32.6 mm to (161.9, 77.5), turned to 90 degrees
- moved R16 31.6 mm to (194.9, 99.7), turned to 270 degrees
- moved J8 30.5 mm to (152.4, 81.3)
- moved D9 29.9 mm to (194.9, 94.6), turned to 270 degrees
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Connections:
- C6 pad 1: /Sheet61A8C81E/12v -> +5V
- U1 pad 38: (no net) -> GND
- U6 pad 3: /Sheet61A8C81E/12v -> +5V
Routing:
- net GND: track 47.4 -> 249.6 mm
- net +3V3: track 0.00 -> 72.1 mm
- net +5V: track 0.00 -> 55.8 mm
- net Net-(R2-Pad2): track 0.00 -> 55.1 mm
- net /Sheet61A8C81E/12v: track 0.00 -> 35.5 mm
- net Net-(C5-Pad1): track 0.00 -> 29.1 mm
- net Net-(R1-Pad2): track 0.00 -> 26.2 mm
- net Net-(D10-Pad1): track 0.00 -> 9.00 mm
- net Net-(D7-Pad2): track 0.00 -> 3.06 mm
- net Net-(D9-Pad2): track 0.00 -> 3.05 mm
- net Net-(D10-Pad2): track 0.00 -> 2.94 mm

Commit message: alimentacion
Parts:
- added Cdes1: 100n, Capacitor_SMD:C_0805_2012Metric_Pad1.18x1.45mm_HandSolder, F.Cu at (203.2, 76.5)
- moved Q3 32.3 mm to (182.9, 113.8), turned to 270 degrees
- moved R13 31.6 mm to (173.7, 116.6)
- moved D7 29.4 mm to (191.8, 97.3), turned to 0 degrees
- moved R14 29.4 mm to (191.8, 102.4), turned to 0 degrees
- moved C6 27.4 mm to (173.7, 108.7), turned to 90 degrees
- moved U5 26.4 mm to (183.1, 97.3), turned to 270 degrees
- moved C5 24.6 mm to (173.7, 99.1)
- moved C7 24.6 mm to (174.2, 83.3)
- moved J8 22.5 mm to (162.7, 101.3)
- moved C8 19.1 mm to (184.2, 73.7), turned to 180 degrees
- moved R15 17.0 mm to (191.6, 80.5), turned to 0 degrees
- moved D9 16.5 mm to (203.5, 80.5)
- moved D8 15.4 mm to (191.8, 85.6), turned to 0 degrees
- moved R2 14.0 mm to (208.3, 107.4)
- moved R1 11.7 mm to (210.3, 81.0)
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Routing:
- net Net-(R2-Pad2): track 55.1 -> 0.00 mm
- net +3V3: track 72.1 -> 19.5 mm
- net +5V: track 55.8 -> 81.8 mm
- net Net-(R1-Pad2): track 26.2 -> 1.26 mm
- net GND: track 249.6 -> 226.5 mm, vias 0 -> 1
- net Net-(C5-Pad1): track 29.1 -> 41.6 mm
- net Net-(D10-Pad1): track 9.00 -> 0.00 mm
- net /Sheet61A8C81E/12v: track 35.5 -> 41.1 mm
- net Net-(D8-Pad2): track 0.00 -> 5.20 mm
- net Net-(D9-Pad2): track 3.05 -> 0.00 mm
- net Net-(D10-Pad2): track 2.94 -> 0.52 mm
- net Net-(D7-Pad2): track 3.06 -> 5.09 mm
- net Net-(J7-Pad2): track 31.7 -> 30.9 mm
- net Net-(J7-Pad3): track 35.5 -> 34.7 mm

Commit message: sensores y cto esp32
Parts:
- SW1, SW2: footprint Button_Switch_SMD:SW_SPST_SKQG_WithStem -> Button_Switch_SMD:SW_SPST_TL3305A
- moved u2 79.9 mm to (241.6, 126.2), turned to 180 degrees
- moved u7 73.7 mm to (227.1, 125.7), turned to 180 degrees
- moved IC1 63.3 mm to (186.2, 130.0), turned to 90 degrees
- moved C1 56.3 mm to (193.8, 128.5)
- moved R9 54.3 mm to (190.0, 123.4), turned to 270 degrees
- moved R3 50.7 mm to (208.5, 118.9)
- moved R7 44.8 mm to (194.1, 123.4), turned to 90 degrees
- moved R8 42.9 mm to (199.4, 130.6), turned to 90 degrees
- moved R10 41.4 mm to (199.1, 123.4), turned to 270 degrees
- moved SW2 40.4 mm to (208.5, 72.6)
- moved TH1 34.3 mm to (210.6, 125.2)
- moved R2 30.0 mm to (209.0, 77.5), turned to 0 degrees
- moved SW1 27.9 mm to (198.1, 72.6), turned to 0 degrees
- moved D10 21.5 mm to (204.0, 91.7), turned to 90 degrees
- moved R17 20.8 mm to (198.8, 94.9), turned to 180 degrees
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Routing:
- net GND: track 226.5 -> 324.1 mm, vias 1 -> 2
- net +5V: track 81.8 -> 168.3 mm, vias 0 -> 4
- net Net-(R2-Pad2): track 0.00 -> 62.3 mm, vias 0 -> 2
- net IO12: track 0.00 -> 52.3 mm
- net +3V3: track 19.5 -> 71.7 mm, vias 0 -> 2
- net IO14: track 0.00 -> 40.6 mm
- net IO2: track 0.00 -> 37.9 mm, vias 0 -> 2
- net Net-(R1-Pad2): track 1.26 -> 31.7 mm
- net Net-(D10-Pad1): track 0.00 -> 23.6 mm, vias 0 -> 2
- net Net-(D10-Pad2): track 0.52 -> 7.31 mm
- net Net-(D9-Pad2): track 0.00 -> 6.11 mm
- net Net-(C1-Pad1): track 0.00 -> 3.45 mm
- net IO33: track 0.00 -> 3.44 mm
- net IO32: track 0.00 -> 3.20 mm

Commit message: PCBs ok
Parts:
- removed C1: 0.1uF, Capacitor_SMD:C_0805_2012Metric_Pad1.18x1.45mm_HandSolder
- removed IC1: BH1750FVI-TR, BH1750:WSOF6
- removed R10, R8, R9: 4.7k, Resistor_SMD:R_0805_2012Metric_Pad1.20x1.40mm_HandSolder
- removed R7: 1k, Resistor_SMD:R_0805_2012Metric_Pad1.20x1.40mm_HandSolder
- added J1: Conn_01x04, Connector_JST:JST_EH_B5B-EH-A_1x05_P2.50mm_Vertical, F.Cu at (197.6, 126.0)
Connections:
- TH1 pad 3: (no net) -> Net-(TH1-Pad3)
- U1 pad 10: (no net) -> Net-(U1-Pad10)
- U1 pad 11: (no net) -> Net-(U1-Pad11)
- U1 pad 12: (no net) -> Net-(U1-Pad12)
- U1 pad 17: (no net) -> Net-(U1-Pad17)
- U1 pad 18: (no net) -> Net-(U1-Pad18)
- U1 pad 19: (no net) -> Net-(U1-Pad19)
- U1 pad 20: (no net) -> Net-(U1-Pad20)
- U1 pad 21: (no net) -> Net-(U1-Pad21)
- U1 pad 22: (no net) -> Net-(U1-Pad22)
- U1 pad 23: (no net) -> Net-(U1-Pad23)
- U1 pad 26: (no net) -> Net-(U1-Pad26)
- U1 pad 27: (no net) -> Net-(U1-Pad27)
- U1 pad 28: (no net) -> Net-(U1-Pad28)
- U1 pad 29: (no net) -> Net-(U1-Pad29)
- U1 pad 30: (no net) -> Net-(U1-Pad30)
- U1 pad 31: (no net) -> Net-(U1-Pad31)
- U1 pad 32: (no net) -> Net-(U1-Pad32)
- U1 pad 33: (no net) -> Net-(U1-Pad33)
- U1 pad 36: (no net) -> Net-(U1-Pad36)
- U1 pad 37: (no net) -> Net-(U1-Pad37)
- U1 pad 4: (no net) -> Net-(U1-Pad4)
- U1 pad 5: (no net) -> Net-(U1-Pad5)
- U1 pad 6: (no net) -> Net-(U1-Pad6)
- U1 pad 7: (no net) -> Net-(U1-Pad7)
- u2 pad 2: (no net) -> Net-(u2-Pad2)
- u7 pad 2: (no net) -> Net-(u7-Pad2)
Routing:
- net IO32: track 3.20 -> 53.0 mm, vias 0 -> 2
- net IO33: track 3.44 -> 49.8 mm, vias 0 -> 2
- net +3V3: track 71.7 -> 116.8 mm, vias 2 -> 3
- net GND: track 324.1 -> 344.1 mm
- net Net-(C1-Pad1): track 3.45 -> 0.00 mm
Other:
- board text added: "Vcc"
