File: Diseño PCB/PCB-ESP32S/PCB-ESP32S.kicad_pcb (KiCad board)
At the start: 2 copper layers, 29 parts, among them J1 Conn_01x04, J7 Screw_Terminal_01x03, J8 Screw_Terminal_01x02, Q3 TIP42C, SW1 SW_DIP_x01, SW2 SW_DIP_x01, U1 ESP-32S, U5 LM7805_TO220, U6 LM1117-3.3, u2 Conn_01x04_Male, u7 Conn_01x04_Male

Commit message: pcv v2
Parts:
- added ?: MountingHole_2.2mm_M2, MountingHole:MountingHole_2.2mm_M2, F.Cu at (243.8, 80.0)
- added ?: MountingHole_2.2mm_M2, MountingHole:MountingHole_2.2mm_M2, F.Cu at (243.8, 125.7)
- added ?: MountingHole_2.2mm_M2, MountingHole:MountingHole_2.2mm_M2, F.Cu at (162.6, 125.7)
- added ?: MountingHole_2.2mm_M2, MountingHole:MountingHole_2.2mm_M2, F.Cu at (162.6, 80.0)
- J1: footprint Connector_JST:JST_EH_B5B-EH-A_1x05_P2.50mm_Vertical -> Connector_JST:JST_GH_BM05B-GHS-TBT_1x05-1MP_P1.25mm_Vertical
- J7: footprint TerminalBlock:TerminalBlock_bornier-3_P5.08mm -> Connector_JST:JST_GH_BM03B-GHS-TBT_1x03-1MP_P1.25mm_Vertical
- TH1: footprint Sensors:DHT22_Temperature_Humidity -> Connector_JST:JST_GH_BM04B-GHS-TBT_1x04-1MP_P1.25mm_Vertical
- moved SW2 39.7 mm to (230.7, 105.6), turned to 0 degrees
- moved R2 33.3 mm to (233.9, 99.6)
- moved u2 26.4 mm to (215.2, 125.8)
- moved u7 25.0 mm to (202.1, 125.7)
- moved D10 20.3 mm to (215.7, 108.3)
- moved C8 18.6 mm to (185.7, 92.2), turned to 90 degrees
- moved R17 18.5 mm to (215.7, 102.5), turned to 90 degrees
- moved R15 18.4 mm to (201.4, 96.1)
- moved TH1 17.0 mm to (227.6, 125.7), turned to 180 degrees
- moved J7 15.3 mm to (230.6, 113.9), turned to 90 degrees
- moved J8 15.3 mm to (173.7, 111.9)
- moved R3 14.2 mm to (222.2, 115.2), turned to 180 degrees
- moved D7 12.9 mm to (200.8, 106.5)
- moved R14 12.7 mm to (200.8, 111.3)
- moved Q3 12.5 mm to (178.9, 125.6), turned to 180 degrees
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Connections:
- J1 pad 2: /BH1750/ADDR -> (no net)
- TH1 pad 3: Net-(TH1-Pad3) -> (no net)
- U1 pad 10: Net-(U1-Pad10) -> (no net)
- U1 pad 11: Net-(U1-Pad11) -> (no net)
- U1 pad 12: Net-(U1-Pad12) -> (no net)
- U1 pad 17: Net-(U1-Pad17) -> (no net)
- U1 pad 18: Net-(U1-Pad18) -> (no net)
- U1 pad 19: Net-(U1-Pad19) -> (no net)
- U1 pad 20: Net-(U1-Pad20) -> (no net)
- U1 pad 21: Net-(U1-Pad21) -> (no net)
- U1 pad 22: Net-(U1-Pad22) -> (no net)
- U1 pad 23: Net-(U1-Pad23) -> (no net)
- U1 pad 26: Net-(U1-Pad26) -> (no net)
- U1 pad 27: Net-(U1-Pad27) -> (no net)
- U1 pad 28: Net-(U1-Pad28) -> (no net)
- U1 pad 29: Net-(U1-Pad29) -> (no net)
- U1 pad 30: Net-(U1-Pad30) -> (no net)
- U1 pad 31: Net-(U1-Pad31) -> (no net)
- U1 pad 32: Net-(U1-Pad32) -> (no net)
- U1 pad 33: Net-(U1-Pad33) -> (no net)
- U1 pad 36: Net-(U1-Pad36) -> (no net)
- U1 pad 37: Net-(U1-Pad37) -> (no net)
- U1 pad 4: Net-(U1-Pad4) -> (no net)
- U1 pad 5: Net-(U1-Pad5) -> (no net)
- U1 pad 6: Net-(U1-Pad6) -> (no net)
- U1 pad 7: Net-(U1-Pad7) -> (no net)
- u2 pad 2: Net-(u2-Pad2) -> (no net)
- u7 pad 2: Net-(u7-Pad2) -> (no net)
Routing:
- net Net-(R2-Pad2): track 62.3 -> 20.1 mm, vias 2 -> 0
- net +3V3: track 116.8 -> 144.1 mm
- net IO12: track 52.3 -> 33.6 mm
- net +5V: track 168.3 -> 150.2 mm, vias 4 -> 3
- net /Sheet61A8C81E/12v: track 41.1 -> 23.0 mm
- net GND: track 344.1 -> 355.9 mm, vias 2 -> 4
- net Net-(J7-Pad2): track 30.9 -> 41.1 mm
- net Net-(C5-Pad1): track 41.6 -> 50.3 mm
- net Net-(R1-Pad2): track 31.7 -> 39.8 mm
- net IO33: track 49.8 -> 57.8 mm, vias 2 -> 0
- net IO32: track 53.0 -> 59.6 mm, vias 2 -> 0
- net IO2: track 37.9 -> 43.4 mm, vias 2 -> 0
- net Net-(D10-Pad1): track 23.6 -> 19.7 mm, vias 2 -> 0
- net Net-(D7-Pad2): track 5.09 -> 8.52 mm
- net Net-(D9-Pad2): track 6.11 -> 2.99 mm
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- added copper zone on B.Cu, net GND
- added copper zone on F.Cu, net GND
Other:
- board outline added: 88.9 x 54.6 mm
- rule trace_min: 0.2 -> 0
- rule via_min_size: 0.4 -> 0.8
- board text removed: "Vcc"

Commit message: mejoras pcb1
Parts:
- removed the ? at (243.8, 80.0)
- removed the ? at (243.8, 125.7)
- removed the ? at (162.6, 125.7)
- removed the ? at (162.6, 80.0)
- added ?: MountingHole_2.2mm_M2, MountingHole:MountingHole_2.2mm_M2, F.Cu at (162.6, 125.1)
- added ?: MountingHole_2.2mm_M2, MountingHole:MountingHole_2.2mm_M2, F.Cu at (243.8, 79.4)
- added ?: MountingHole_2.2mm_M2, MountingHole:MountingHole_2.2mm_M2, F.Cu at (243.8, 125.1)
- added ?: MountingHole_2.2mm_M2, MountingHole:MountingHole_2.2mm_M2, F.Cu at (162.6, 79.4)
- SW1: value SW_DIP_x01 -> SW_DIP_x02
- moved R8 2.17 mm to (222.2, 113.0)
- renumbered C5 to C2, C7 to C3, C6 to C4, C8 to C5, D9 to D1, D10 to D2, D7 to D3, D8 to D4, J7 to J1, J8 to J2, J1 to J3, u7 to J4, u2 to J5, Q3 to Q1, R16 to R2, R2 to R3, R17 to R4, R13 to R5, R14 to R6, R15 to R7, R3 to R8, U5 to U2, U6 to U3
Routing:
- net IO2: track 43.4 -> 38.7 mm
- net +3V3: track 144.1 -> 147.3 mm
- net +5V: track 150.2 -> 151.5 mm

Commit message: dos pcb finalizadas
Parts:
- removed the ? at (162.6, 125.1)
- removed the ? at (243.8, 79.4)
- removed the ? at (243.8, 125.1)
- removed the ? at (162.6, 79.4)
- added ?: MountingHole_2.2mm_M2, MountingHole:MountingHole_2.2mm_M2, F.Cu at (174.0, 78.7)
- added ?: MountingHole_2.2mm_M2, MountingHole:MountingHole_2.2mm_M2, F.Cu at (238.8, 125.7)
- added ?: MountingHole_2.2mm_M2, MountingHole:MountingHole_2.2mm_M2, F.Cu at (238.8, 78.7)
- added ?: MountingHole_2.2mm_M2, MountingHole:MountingHole_2.2mm_M2, F.Cu at (174.0, 125.7)
- R5: footprint Resistor_SMD:R_0805_2012Metric_Pad1.20x1.40mm_HandSolder -> Resistor_SMD:R_1210_3225Metric_Pad1.30x2.65mm_HandSolder
- moved Q1 7.90 mm to (174.0, 119.4), turned to 90 degrees
- moved C2 5.75 mm to (174.2, 91.4)
- moved J2 5.02 mm to (174.2, 106.9)
- moved R5 2.81 mm to (178.8, 115.8), turned to 270 degrees
- moved C3 2.28 mm to (180.3, 82.5)
Routing:
- net GND: track 355.9 -> 340.8 mm
- net /Sheet61A8C81E/12v: track 23.0 -> 10.6 mm
- net +5V: track 151.5 -> 147.2 mm
- net Net-(C2-Pad1): track 50.3 -> 51.6 mm
Other:
- board size 88.9 x 54.6 mm -> 72.4 x 54.6 mm
