File: Diseño PCB/PCB-ESP32S/PCB-ESP32S.kicad_pcb (KiCad board)
At the start: 2 copper layers, 72.4 x 54.6 mm, 33 parts, among them J1 Screw_Terminal_01x03, J2 Screw_Terminal_01x02, J3 Conn_01x04, J4 Conn_01x04_Male, J5 Conn_01x04_Male, Q1 TIP42C, SW1 SW_DIP_x02, SW2 SW_DIP_x01, U1 ESP-32S, U2 LM7805_TO220, U3 LM1117-3.3

Commit message: edicion true hole
Parts:
- J1: footprint Connector_JST:JST_GH_BM03B-GHS-TBT_1x03-1MP_P1.25mm_Vertical -> Connector_JST:JST_EH_B3B-EH-A_1x03_P2.50mm_Vertical
- J3: footprint Connector_JST:JST_GH_BM05B-GHS-TBT_1x05-1MP_P1.25mm_Vertical -> Connector_JST:JST_EH_B5B-EH-A_1x05_P2.50mm_Vertical
- J4, J5, TH1: footprint Connector_JST:JST_GH_BM04B-GHS-TBT_1x04-1MP_P1.25mm_Vertical -> Connector_JST:JST_EH_B4B-EH-A_1x04_P2.50mm_Vertical
- moved TH1 5.46 mm to (233.0, 125.7)
- moved J1 4.00 mm to (232.4, 117.5)
- moved J5 3.28 mm to (218.4, 125.7)
- moved J4 1.78 mm to (203.8, 125.7)
- moved J3 0.34 mm to (189.9, 125.7)
Routing:
- net GND: track 340.8 -> 352.0 mm
- net +5V: track 147.2 -> 156.2 mm, vias 3 -> 1
- net IO14: track 41.6 -> 47.7 mm
- net +3V3: track 147.3 -> 153.1 mm
- net IO32: track 59.6 -> 64.6 mm
- net IO33: track 57.8 -> 62.3 mm
- net IO2: track 38.7 -> 42.1 mm
- net IO12: track 33.6 -> 34.8 mm
- net Net-(J1-Pad2): track 41.1 -> 41.9 mm
- net Net-(J1-Pad3): track 36.6 -> 35.8 mm

Commit message: PCB caca super caca2
Routing:
- net +3V3: track 153.1 -> 166.6 mm, vias 3 -> 5
- net +5V: track 156.2 -> 168.4 mm, vias 1 -> 3
- net GND: track 352.0 -> 363.5 mm, vias 4 -> 7
- net Net-(C2-Pad1): track 51.6 -> 57.2 mm, vias 0 -> 2
- net /Sheet61A8C81E/12v: track 10.6 -> 15.5 mm, vias 0 -> 1
- net Net-(J1-Pad3): track 35.8 -> 37.4 mm, vias 0 -> 1
- net IO2: track 42.1 -> 43.1 mm, vias 0 -> 1
- net IO12: track 34.8 -> 33.8 mm, vias 0 -> 1
- net Net-(J1-Pad2): track 41.9 -> 42.3 mm, vias 0 -> 1
- net IO33: track 62.3 -> 61.9 mm, vias 0 -> 1
- net IO14: vias 0 -> 1
- net IO32: vias 0 -> 1
