File: Diseño PCB/PCB-ESP32S/pines_sensor2.sch (KiCad schematic (older format))
At the start: 1 part, among them u2 Conn_01x04_Male

Commit message: mejoras pcb1
Parts:
- renumbered u2 to J5
Changed lines of the file:
@@
 P 4100 2050
 AR Path="/61A90AD5/61E2ED63" Ref="u?"  Part="1"
-AR Path="/61E0EDBD/61E2ED63" Ref="u2"  Part="1"
-F 0 "u2" H 4208 2331 50  0000 C CNN
+AR Path="/61E0EDBD/61E2ED63" Ref="J5"  Part="1"
+F 0 "J5" H 4208 2331 50  0000 C CNN
 F 1 "Conn_01x04_Male" H 4208 2240 50  0000 C CNN
 F 2 "Connector_JST:JST_GH_BM04B-GHS-TBT_1x04-1MP_P1.25mm_Vertical" H 4100 2050 50  0001 C CNN

Commit message: edicion true hole
Parts:
- J5: footprint Connector_JST:JST_GH_BM04B-GHS-TBT_1x04-1MP_P1.25mm_Vertical -> Connector_JST:JST_EH_B4B-EH-A_1x04_P2.50mm_Vertical
Changed lines of the file:
@@
 F 0 "J5" H 4208 2331 50  0000 C CNN
 F 1 "Conn_01x04_Male" H 4208 2240 50  0000 C CNN
-F 2 "Connector_JST:JST_GH_BM04B-GHS-TBT_1x04-1MP_P1.25mm_Vertical" H 4100 2050 50  0001 C CNN
+F 2 "Connector_JST:JST_EH_B4B-EH-A_1x04_P2.50mm_Vertical" H 4100 2050 50  0001 C CNN
 F 3 "~" H 4100 2050 50  0001 C CNN
 	1    4100 2050
