File: Diseño PCB/PCB-ESP32S - reles/PCB-ESP32S.kicad_pcb (KiCad board)
At the start: 2 copper layers, 39 parts, among them J1 Screw_Terminal_01x03, J3 Screw_Terminal_01x03, J7 Screw_Terminal_01x03, J8 Screw_Terminal_01x02, K1 SRD-05VDC-SL-C, K2 SRD-05VDC-SL-C, Q1 MMBT2222A, Q2 MMBT2222A, Q3 TIP42C, SW1 SW_DIP_x01, SW2 SW_DIP_x01, U1 ESP-32S, U3 PC817, U4 PC817, U5 LM7805_TO220, U6 LM1117-3.3

Commit message: Pines sensores
Parts:
- moved U1 120.6 mm to (255.3, 48.3)
- moved C5 99.9 mm to (319.1, 109.0)
- moved C7 99.9 mm to (319.1, 117.1)
- moved D1 99.9 mm to (201.9, 125.7)
- moved D3 99.9 mm to (195.3, 130.4)
- moved K1 99.9 mm to (265.7, 113.4)
- moved K2 99.9 mm to (287.0, 113.4)
- moved R4 99.9 mm to (212.7, 119.8)
- moved C8 99.9 mm to (305.3, 115.6)
- moved D10 99.9 mm to (304.7, 125.9)
- moved D2 99.9 mm to (215.4, 113.1)
- moved D4 99.9 mm to (187.9, 131.2)
- moved D7 99.9 mm to (310.8, 115.5)
- moved D9 99.9 mm to (309.5, 125.9)
- moved J1 99.9 mm to (186.1, 124.4)
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Connections:
- D1 pad 1: (no net) -> /ModulosReles/GPIO1
- D3 pad 1: (no net) -> /ModulosReles/GPIO2
- R4 pad 1: (no net) -> Net-(R4-Pad1)
- R5 pad 1: (no net) -> /ModulosReles/VESP32
- U1 pad 10: (no net) -> Net-(U1-Pad10)
- U1 pad 11: (no net) -> Net-(U1-Pad11)
- U1 pad 12: (no net) -> Net-(U1-Pad12)
- U1 pad 13: (no net) -> Net-(U1-Pad13)
- U1 pad 14: (no net) -> Net-(U1-Pad14)
- U1 pad 17: (no net) -> Net-(U1-Pad17)
- U1 pad 18: (no net) -> Net-(U1-Pad18)
- U1 pad 19: (no net) -> Net-(U1-Pad19)
- U1 pad 20: (no net) -> Net-(U1-Pad20)
- U1 pad 21: (no net) -> Net-(U1-Pad21)
- U1 pad 22: (no net) -> Net-(U1-Pad22)
- U1 pad 23: (no net) -> Net-(U1-Pad23)
- U1 pad 24: (no net) -> Net-(U1-Pad24)
- U1 pad 26: (no net) -> Net-(U1-Pad26)
- U1 pad 27: (no net) -> Net-(U1-Pad27)
- U1 pad 28: (no net) -> Net-(U1-Pad28)
- U1 pad 29: (no net) -> Net-(U1-Pad29)
- U1 pad 30: (no net) -> Net-(U1-Pad30)
- U1 pad 31: (no net) -> Net-(U1-Pad31)
- U1 pad 32: (no net) -> Net-(U1-Pad32)
- U1 pad 33: (no net) -> Net-(U1-Pad33)
- U1 pad 36: (no net) -> Net-(U1-Pad36)
- U1 pad 37: (no net) -> Net-(U1-Pad37)
- U1 pad 38: (no net) -> Net-(U1-Pad38)
- U1 pad 4: (no net) -> Net-(U1-Pad4)
- U1 pad 5: (no net) -> Net-(U1-Pad5)
- U1 pad 6: (no net) -> Net-(U1-Pad6)
- U1 pad 7: (no net) -> Net-(U1-Pad7)
- U1 pad 8: (no net) -> Net-(U1-Pad8)
- U1 pad 9: (no net) -> Net-(U1-Pad9)

Commit message: PCB2
Parts:
- moved C5 211.7 mm to (117.2, 45.5)
- moved C7 211.7 mm to (117.2, 53.6)
- moved C6 203.9 mm to (129.5, 57.1)
- moved D7 198.6 mm to (118.1, 67.3)
- moved J8 191.4 mm to (129.5, 34.3)
- moved C8 179.6 mm to (128.6, 83.8)
- moved D9 148.4 mm to (191.8, 35.6), turned to 180 degrees
- moved R16 120.8 mm to (185.4, 22.9)
- moved D10 112.6 mm to (219.7, 52.1)
- moved R6 94.4 mm to (282.2, 83.8)
- moved Q2 88.7 mm to (188.0, 73.7), turned to 90 degrees
- moved K2 86.8 mm to (204.5, 86.4)
- moved U3 84.1 mm to (276.9, 76.2), turned to 270 degrees
- moved D1 74.3 mm to (242.6, 63.5), turned to 270 degrees
- moved R17 73.7 mm to (226.1, 54.6)
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Connections:
- net /ModulosReles/VCC_source renamed +12V
- D1 pad 1: /ModulosReles/GPIO1 -> IO12
- D3 pad 1: /ModulosReles/GPIO2 -> IO14
- R5 pad 1: /ModulosReles/VESP32 -> +5V
- U1 pad 13: Net-(U1-Pad13) -> IO14
- U1 pad 14: Net-(U1-Pad14) -> IO12
Routing:
- net GND: track 0.00 -> 61.1 mm
- net Net-(J7-Pad3): track 0.00 -> 35.3 mm
- net Net-(J7-Pad2): track 0.00 -> 33.0 mm
- net /ModulosReles/NO: track 0.00 -> 3.10 mm
- net +12V: track 0.00 -> 1.39 mm
- net IO12: track 0.00 -> 0.89 mm

Commit message: PCB reles
Parts:
- added Cdes1: 100n, Capacitor_SMD:C_0805_2012Metric_Pad1.18x1.45mm_HandSolder, F.Cu at (207.0, 15.2)
- moved Q2 39.8 mm to (227.6, 77.7), turned to 0 degrees
- moved J1 39.4 mm to (259.1, 110.7), turned to 180 degrees
- moved J3 30.7 mm to (212.9, 109.7), turned to 180 degrees
- moved U3 28.5 mm to (248.4, 78.0), turned to 0 degrees
- moved R6 20.8 mm to (261.6, 80.5)
- moved K1 18.7 mm to (254.0, 93.3)
- moved SW2 18.6 mm to (204.0, 28.4)
- moved D10 18.6 mm to (210.3, 36.1)
- moved R17 18.6 mm to (216.7, 38.6)
- moved R2 18.6 mm to (206.8, 23.4)
- moved D1 17.0 mm to (241.6, 80.5), turned to 0 degrees
- moved R5 14.9 mm to (241.6, 78.0), turned to 0 degrees
- moved D2 12.5 mm to (260.1, 71.6)
- moved D4 8.63 mm to (214.6, 70.6), turned to 0 degrees
- moved K2 8.30 mm to (207.8, 94.0), turned to 180 degrees
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Connections:
- J1 pad 1: /ModulosReles/NO -> /ModulosReles/NO2
- J1 pad 2: /ModulosReles/C -> /ModulosReles/C2
- J1 pad 3: /ModulosReles/NC -> /ModulosReles/NC2
- K1 pad COM: /ModulosReles/C -> /ModulosReles/C2
- K1 pad NC: /ModulosReles/NC -> /ModulosReles/NC2
- K1 pad NO: /ModulosReles/NO -> /ModulosReles/NO2
- R4 pad 1: Net-(R4-Pad1) -> +5V
Routing:
- net GND: track 61.1 -> 194.4 mm, vias 0 -> 2
- net +12V: track 1.39 -> 113.4 mm
- net IO14: track 0.00 -> 81.3 mm
- net IO12: track 0.89 -> 44.7 mm
- net /ModulosReles/C: track 0.00 -> 43.1 mm
- net /ModulosReles/C2: track 0.00 -> 40.3 mm
- net Net-(D2-Pad2): track 0.00 -> 33.2 mm, vias 0 -> 1
- net Net-(D4-Pad2): track 0.17 -> 32.8 mm, vias 0 -> 1
- net /ModulosReles/NO: track 3.10 -> 33.4 mm
- net /ModulosReles/NO2: track 0.00 -> 30.1 mm
- net /ModulosReles/NC2: track 0.00 -> 13.1 mm
- net /ModulosReles/NC: track 0.00 -> 12.3 mm
- net Net-(Q1-Pad1): track 0.24 -> 9.56 mm
- net Net-(Q2-Pad1): track 0.00 -> 8.40 mm
- net Net-(R5-Pad2): track 0.00 -> 5.86 mm
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
Commit message: PCBs ok
Parts:
- SW1, SW2: footprint Button_Switch_SMD:SW_SPST_SKQG_WithStem -> Button_Switch_SMD:SW_SPST_TL3305A
- moved C8 78.5 mm to (179.8, 24.4), turned to 180 degrees
- moved D7 77.1 mm to (193.5, 51.3)
- moved D8 60.2 mm to (192.8, 38.1)
- moved C7 55.8 mm to (169.7, 34.8), turned to 90 degrees
- moved C5 53.5 mm to (169.7, 55.9), turned to 90 degrees
- moved R14 52.5 mm to (193.8, 57.4)
- moved R15 52.0 mm to (192.8, 33.3)
- moved Q3 42.5 mm to (184.4, 72.9), turned to 270 degrees
- moved C6 42.0 mm to (170.7, 65.8), turned to 90 degrees
- moved U5 38.6 mm to (184.4, 52.3), turned to 270 degrees
- moved J8 36.3 mm to (156.0, 59.2), turned to 90 degrees
- moved U6 31.7 mm to (185.2, 38.1), turned to 90 degrees
- moved R16 27.6 mm to (203.5, 43.7), turned to 180 degrees
- moved Cdes1 23.1 mm to (203.5, 38.1), turned to 180 degrees
- moved D9 21.1 mm to (212.6, 38.9), turned to 270 degrees
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Connections:
- C6 pad 1: /Sheet61A8C81E/12v -> +5V
- U6 pad 3: /Sheet61A8C81E/12v -> +5V
Routing:
- net GND: track 194.4 -> 402.2 mm, vias 2 -> 0
- net +5V: track 0.00 -> 180.6 mm, vias 0 -> 2
- net +3V3: track 0.00 -> 98.7 mm, vias 0 -> 2
- net Net-(R2-Pad2): track 0.00 -> 89.8 mm, vias 0 -> 2
- net Net-(C5-Pad1): track 0.00 -> 57.0 mm
- net Net-(R1-Pad2): track 0.00 -> 54.3 mm
- net Net-(D10-Pad1): track 0.00 -> 48.8 mm, vias 0 -> 2
- net /Sheet61A8C81E/12v: track 0.00 -> 45.0 mm
- net Net-(D10-Pad2): track 0.00 -> 10.4 mm
- net Net-(D9-Pad2): track 0.00 -> 9.72 mm
- net Net-(D7-Pad2): track 0.00 -> 6.21 mm
- net Net-(D8-Pad2): track 0.00 -> 4.87 mm

Commit message: PCB reles - GND plano
Parts:
- moved R13 36.5 mm to (203.5, 57.4)
- moved J1 36.2 mm to (271.5, 76.7), turned to 270 degrees
- moved J3 30.3 mm to (224.5, 81.8), turned to 270 degrees
- moved C6 26.8 mm to (188.5, 45.7)
- moved C5 26.6 mm to (194.6, 46.5)
- moved J8 25.9 mm to (181.9, 60.5)
- moved C7 24.9 mm to (194.6, 34.5)
- moved U5 22.5 mm to (204.5, 42.2)
- moved D7 22.0 mm to (214.9, 46.0)
- moved R14 22.0 mm to (215.2, 52.1)
- moved D8 21.4 mm to (214.1, 36.1)
- moved R18 21.4 mm to (214.1, 31.2)
- moved U6 21.4 mm to (204.5, 29.0), turned to 270 degrees
- moved R17 20.4 mm to (223.5, 45.7)
- moved Q3 20.4 mm to (194.8, 55.4)
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- renumbered R15 to R18
Connections:
- J8 pad 1: /Sheet61A8C81E/12v -> +12V
- Q3 pad 3: /Sheet61A8C81E/12v -> +12V
- R13 pad 1: /Sheet61A8C81E/12v -> +12V
Routing:
- net GND: track 402.2 -> 345.2 mm
- net +5V: track 180.6 -> 127.2 mm
- net +12V: track 113.4 -> 163.1 mm
- net /Sheet61A8C81E/12v: track 45.0 -> 0.00 mm
- net Net-(C5-Pad1): track 57.0 -> 23.2 mm
- net /ModulosReles/C: track 43.1 -> 10.8 mm
- net /ModulosReles/C2: track 40.3 -> 11.1 mm
- net Net-(D10-Pad1): track 48.8 -> 20.6 mm
- net +3V3: track 98.7 -> 71.2 mm
- net Net-(R1-Pad2): track 54.3 -> 34.8 mm
- net Net-(R2-Pad2): track 89.8 -> 70.7 mm
- net /ModulosReles/NC2: track 13.1 -> 31.0 mm
- net /ModulosReles/NC: track 12.3 -> 28.9 mm
- net IO12: track 44.7 -> 31.4 mm
- net IO14: track 81.3 -> 69.8 mm, vias 0 -> 2
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- added copper zone on B.Cu, net GND
- added copper zone on F.Cu, net GND
Other:
- board outline added: 109.2 x 83.8 mm

Commit message: PCB reles
Parts:
- added REF**: MountingHole_2.2mm_M2, MountingHole:MountingHole_2.2mm_M2, F.Cu at (285.8, 91.4)
- added REF**: MountingHole_2.2mm_M2, MountingHole:MountingHole_2.2mm_M2, F.Cu at (198.1, 91.4)
- added REF**: MountingHole_2.2mm_M2, MountingHole:MountingHole_2.2mm_M2, F.Cu at (198.1, 21.6)
- added REF**: MountingHole_2.2mm_M2, MountingHole:MountingHole_2.2mm_M2, F.Cu at (285.8, 21.6)
- J7: footprint TerminalBlock:TerminalBlock_bornier-3_P5.08mm -> Connector_JST:JST_GH_BM03B-GHS-TBT_1x03-1MP_P1.25mm_Vertical
- moved SW2 44.0 mm to (267.3, 47.9), turned to 0 degrees
- moved R2 38.7 mm to (268.9, 41.6)
- moved C6 35.5 mm to (223.2, 52.9)
- moved K2 31.8 mm to (237.2, 82.7)
- moved R17 30.4 mm to (253.9, 44.9), turned to 90 degrees
- moved C8 29.6 mm to (223.8, 34.6), turned to 90 degrees
- moved Cdes1 28.3 mm to (247.0, 21.0), turned to 90 degrees
- moved R16 27.7 mm to (242.3, 21.0), turned to 90 degrees
- moved J8 26.5 mm to (207.1, 52.2)
- moved R18 26.5 mm to (239.3, 39.2)
- moved U5 26.3 mm to (230.0, 48.3)
- moved U6 26.0 mm to (229.9, 34.3)
- moved D8 25.2 mm to (239.2, 34.3)
- moved D10 24.2 mm to (253.8, 50.7)
- moved D7 22.9 mm to (237.6, 49.0)
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Routing:
- net Net-(R2-Pad2): track 70.7 -> 19.6 mm, vias 2 -> 0
- net Net-(C5-Pad1): track 23.2 -> 50.5 mm
- net +5V: track 127.2 -> 102.7 mm, vias 2 -> 0
- net IO14: track 69.8 -> 92.7 mm
- net +12V: track 163.1 -> 140.4 mm, vias 0 -> 1
- net GND: track 345.2 -> 325.0 mm, vias 0 -> 2
- net +3V3: track 71.2 -> 90.3 mm, vias 2 -> 3
- net /ModulosReles/C: track 10.8 -> 27.4 mm
- net /ModulosReles/NC: track 28.9 -> 13.7 mm
- net /ModulosReles/NO: track 29.1 -> 14.8 mm
- net Net-(D1-Pad2): track 5.83 -> 14.4 mm
- net Net-(J7-Pad2): track 33.0 -> 40.6 mm
- net IO12: track 31.4 -> 24.1 mm
- net Net-(D4-Pad2): track 33.4 -> 27.0 mm, vias 1 -> 0
- net Net-(D9-Pad2): track 8.09 -> 3.09 mm
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Other:
- board outline removed

Commit message: dos pcb finalizadas
Parts:
- removed REF** (x4): MountingHole_2.2mm_M2, MountingHole:MountingHole_2.2mm_M2
- added ?: MountingHole_2.2mm_M2, MountingHole:MountingHole_2.2mm_M2, F.Cu at (176.4, 68.0)
- added ?: MountingHole_2.2mm_M2, MountingHole:MountingHole_2.2mm_M2, F.Cu at (104.0, 68.0)
- added ?: MountingHole_2.2mm_M2, MountingHole:MountingHole_2.2mm_M2, F.Cu at (176.4, 136.6)
- added ?: MountingHole_2.2mm_M2, MountingHole:MountingHole_2.2mm_M2, F.Cu at (104.0, 136.6)
- R5: renamed from R13; footprint Resistor_SMD:R_0805_2012Metric_Pad1.20x1.40mm_HandSolder -> Resistor_SMD:R_1210_3225Metric_Pad1.30x2.65mm_HandSolder
- moved Q3 127.3 mm to (119.0, 112.2), turned to 180 degrees
- moved J3 126.2 mm to (164.2, 125.7)
- moved Q2 123.7 mm to (147.8, 106.4), turned to 180 degrees
- moved D7 122.7 mm to (147.5, 116.4), turned to 180 degrees
- moved J4 122.1 mm to (111.3, 136.4), turned to 90 degrees
- moved K1 121.8 mm to (147.5, 129.7), turned to 270 degrees
- moved K2 119.7 mm to (127.2, 130.0), turned to 270 degrees
- moved R9 115.4 mm to (152.7, 110.9)
- moved D8 113.7 mm to (127.2, 116.9), turned to 180 degrees
- moved R5 113.6 mm to (110.5, 105.4)
- moved D4 113.4 mm to (136.0, 81.3)
- moved R7 113.4 mm to (136.1, 86.1)
- moved U2 112.0 mm to (128.4, 95.3)
- moved R2 111.9 mm to (140.7, 68.0)
- moved C3 111.9 mm to (112.6, 73.2)
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- renumbered C5 to C2, C7 to C3, C6 to C4, C8 to C5, D9 to D1, D10 to D2, D7 to D3, D8 to D4, D1 to D5, D3 to D6, D2 to D7, D4 to D8, J7 to J1, J1 to J3, J3 to J4, Q3 to Q1, Q1 to Q2, Q2 to Q3, R4 to R10, R16 to R2, R2 to R3, R17 to R4, R14 to R6, R18 to R7, R5 to R8, R6 to R9, U5 to U2, U6 to U3, U3 to U4, U4 to U5
Connections:
- U1 pad 10: Net-(U1-Pad10) -> (no net)
- U1 pad 11: Net-(U1-Pad11) -> (no net)
- U1 pad 12: Net-(U1-Pad12) -> (no net)
- U1 pad 17: Net-(U1-Pad17) -> (no net)
- U1 pad 18: Net-(U1-Pad18) -> (no net)
- U1 pad 19: Net-(U1-Pad19) -> (no net)
- U1 pad 20: Net-(U1-Pad20) -> (no net)
- U1 pad 21: Net-(U1-Pad21) -> (no net)
- U1 pad 22: Net-(U1-Pad22) -> (no net)
- U1 pad 23: Net-(U1-Pad23) -> (no net)
- U1 pad 24: Net-(U1-Pad24) -> (no net)
- U1 pad 26: Net-(U1-Pad26) -> (no net)
- U1 pad 27: Net-(U1-Pad27) -> (no net)
- U1 pad 28: Net-(U1-Pad28) -> (no net)
- U1 pad 29: Net-(U1-Pad29) -> (no net)
- U1 pad 30: Net-(U1-Pad30) -> (no net)
- U1 pad 31: Net-(U1-Pad31) -> (no net)
- U1 pad 32: Net-(U1-Pad32) -> (no net)
- U1 pad 33: Net-(U1-Pad33) -> (no net)
- U1 pad 36: Net-(U1-Pad36) -> (no net)
- U1 pad 37: Net-(U1-Pad37) -> (no net)
- U1 pad 38: Net-(U1-Pad38) -> GND
- U1 pad 4: Net-(U1-Pad4) -> (no net)
- U1 pad 5: Net-(U1-Pad5) -> (no net)
- U1 pad 6: Net-(U1-Pad6) -> (no net)
- U1 pad 7: Net-(U1-Pad7) -> (no net)
- U1 pad 8: Net-(U1-Pad8) -> (no net)
- U1 pad 9: Net-(U1-Pad9) -> (no net)
Routing:
- net IO14: track 92.7 -> 13.3 mm, vias 2 -> 0
- net +5V: track 102.7 -> 148.0 mm, vias 0 -> 2
- net /ModulosReles/NC2: track 29.0 -> 10.8 mm
- net Net-(D6-Pad2): track 4.28 -> 17.1 mm
- net /ModulosReles/NC: track 13.7 -> 26.0 mm
- net GND: track 325.0 -> 337.3 mm
- net +12V: track 140.4 -> 128.6 mm, vias 1 -> 0
- net Net-(D5-Pad2): track 14.4 -> 4.23 mm
- net Net-(D2-Pad1): track 19.9 -> 10.8 mm
- net Net-(Q2-Pad1): track 4.56 -> 13.5 mm
- net Net-(D8-Pad2): track 27.0 -> 18.6 mm
- net /ModulosReles/C2: track 15.4 -> 23.6 mm
- net Net-(R10-Pad2): track 4.29 -> 11.5 mm
- net /ModulosReles/C: track 27.4 -> 22.3 mm
- net Net-(D7-Pad2): track 30.9 -> 25.8 mm, vias 1 -> 0
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Other:
- board outline added: 80 x 76.2 mm
