File: Diseño PCB/PCB-ESP32S - reles/PCB-ESP32S.kicad_pcb (KiCad board)
At the start: 2 copper layers, 80 x 76.2 mm, 44 parts, among them J1 Screw_Terminal_01x03, J3 Screw_Terminal_01x03, J4 Screw_Terminal_01x03, J8 Screw_Terminal_01x02, K1 SRD-05VDC-SL-C, K2 SRD-05VDC-SL-C, Q1 TIP42C, Q2 MMBT2222A, Q3 MMBT2222A, SW1 SW_DIP_x01, SW2 SW_DIP_x01, U1 ESP-32S, U2 LM7805_TO220, U3 LM1117-3.3, U4 PC817, U5 PC817

Commit message: primer cambio super problema
Parts:
- moved ? 14.8 mm to (104.2, 121.8)
- moved J4 1.65 mm to (111.3, 134.8)
Routing:
- net +12V: track 128.6 -> 172.2 mm, vias 0 -> 3
- net GND: track 345.5 -> 369.7 mm, vias 2 -> 5
- net Net-(R8-Pad2): track 3.42 -> 27.1 mm, vias 0 -> 1
- net /ModulosReles/NO2: track 26.9 -> 49.7 mm
- net +3V3: track 92.5 -> 113.7 mm, vias 3 -> 4
- net /ModulosReles/NC: track 26.0 -> 46.6 mm
- net Net-(C2-Pad1): track 53.2 -> 73.3 mm, vias 0 -> 2
- net +5V: track 148.0 -> 166.4 mm, vias 2 -> 3
- net Net-(D7-Pad2): track 25.8 -> 40.2 mm, vias 0 -> 1
- net Net-(R9-Pad1): track 9.95 -> 24.1 mm, vias 0 -> 1
- net Net-(D8-Pad2): track 18.6 -> 30.9 mm, vias 0 -> 1
- net Net-(R10-Pad2): track 11.5 -> 23.1 mm, vias 0 -> 1
- net Net-(R11-Pad1): track 5.41 -> 17.0 mm, vias 0 -> 1
- net Net-(J1-Pad3): track 41.3 -> 51.0 mm, vias 0 -> 1
- net Net-(D6-Pad2): track 17.1 -> 26.1 mm, vias 0 -> 1
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