File: Diseño PCB/PCB-ESP32S - reles/PCB-ESP32S.kicad_pcb (KiCad board)
At the start: 2 copper layers, 80 x 76.2 mm, 44 parts, among them J1 Screw_Terminal_01x03, J3 Screw_Terminal_01x03, J4 Screw_Terminal_01x03, J8 Screw_Terminal_01x02, K1 SRD-05VDC-SL-C, K2 SRD-05VDC-SL-C, Q1 TIP42C, Q2 MMBT2222A, Q3 MMBT2222A, SW1 SW_DIP_x01, SW2 SW_DIP_x01, U1 ESP-32S, U2 LM7805_TO220, U3 LM1117-3.3, U4 PC817, U5 PC817

Commit message: PCB relés, te lo juro por Dieguito Maradona :''v
Parts:
- J1: footprint Connector_JST:JST_GH_BM03B-GHS-TBT_1x03-1MP_P1.25mm_Vertical -> Connector_JST:JST_EH_B3B-EH-A_1x03_P2.50mm_Vertical
- moved J1 7.62 mm to (168.2, 111.6)
Routing:
- net GND: track 337.3 -> 345.5 mm
- net Net-(J1-Pad2): track 40.4 -> 47.2 mm
- net Net-(J1-Pad3): track 36.9 -> 41.3 mm
