File: Diseño PCB/PCB-ESP32S - reles/alimentacion.sch (KiCad schematic (older format))
At the start: 13 parts, among them J8 Screw_Terminal_01x02, Q3 TIP42C, U5 LM7805_TO220, U6 LM1117-3.3

Commit message: PCBs ok
Connections:
- net 12v: no longer C6.1, U6.3 (VI)
- net 5V: now also C6.1, U6.3 (VI)
Changed lines of the file:
@@
 $EndComp
 Wire Wire Line
-	5250 2950 5750 2950
+	5250 2950 5600 2950
 $Comp
 L pspice:CAP C6
@@
 Wire Wire Line
 	3500 2900 3600 2900
-Wire Wire Line
-	3100 2900 3100 4450
-Wire Wire Line
-	3100 4450 3600 4450
-Connection ~ 3600 4450
 Connection ~ 3600 3850
 Connection ~ 3600 5400
@@
 Text HLabel 2900 2900 0    50   Input ~ 0
 12v
+Wire Wire Line
+	5600 2950 5600 4150
+Wire Wire Line
+	5600 4150 3600 4150
+Wire Wire Line
+	3600 4150 3600 4450
+Connection ~ 5600 2950
+Wire Wire Line
+	5600 2950 5750 2950
+Connection ~ 3600 4450
 $EndSCHEMATC

Commit message: pcv v2
Parts:
- renumbered R15 to R18
Changed lines of the file:
@@
 	1    0    0    -1
 $EndComp
-Wire Wire Line
-	5250 2950 5600 2950
 $Comp
 L pspice:CAP C6
@@
 $EndComp
 $Comp
-L Device:R R15
+L Device:R R18
 U 1 1 61A875B1
 P 5250 4800
-F 0 "R15" H 5320 4846 50  0000 L CNN
+F 0 "R18" H 5320 4846 50  0000 L CNN
 F 1 "470" H 5320 4755 50  0000 L CNN
 F 2 "Resistor_SMD:R_0805_2012Metric_Pad1.20x1.40mm_HandSolder" V 5180 4800 50  0001 C CNN
@@
 Wire Wire Line
 	5250 4450 5250 4650
-Wire Wire Line
-	5250 5000 5250 4950
-Wire Wire Line
-	5250 4450 5750 4450
-Connection ~ 5250 4450
 $Comp
 L Regulator_Linear:LM1117-3.3 U6
@@
 Wire Wire Line
 	3000 5400 3600 5400
-Text HLabel 5750 2950 3    50   Input ~ 0
+Text HLabel 6100 2950 3    50   Input ~ 0
 5V
 Text HLabel 5750 4450 3    50   Input ~ 0
@@
 12v
 Wire Wire Line
-	5600 2950 5600 4150
+	3600 4150 3600 4450
+Connection ~ 3600 4450
 Wire Wire Line
-	5600 4150 3600 4150
+	5250 5000 5250 4950
+Connection ~ 5250 4450
 Wire Wire Line
-	3600 4150 3600 4450
-Connection ~ 5600 2950
+	6000 4150 6000 2950
+Connection ~ 6000 2950
 Wire Wire Line
-	5600 2950 5750 2950
-Connection ~ 3600 4450
+	6000 2950 6100 2950
+Wire Wire Line
+	3600 4150 6000 4150
+Wire Wire Line
+	5250 4450 5750 4450
+Wire Wire Line
+	5250 2950 6000 2950
 $EndSCHEMATC

Commit message: PCB reles - GND plano
Connections:
- net 12v renamed +12V
Changed lines of the file:
@@
 	3000 4350 3000 5400
 Text HLabel 2900 2900 0    50   Input ~ 0
-12v
++12V
 Wire Wire Line
 	3600 4150 3600 4450

Commit message: dos pcb finalizadas
Parts:
- R5: renamed from R13; footprint Resistor_SMD:R_0805_2012Metric_Pad1.20x1.40mm_HandSolder -> Resistor_SMD:R_1210_3225Metric_Pad1.30x2.65mm_HandSolder
- renumbered C5 to C2, C7 to C3, C6 to C4, C8 to C5, D7 to D3, D8 to D4, Q3 to Q1, R14 to R6, R18 to R7, U5 to U2, U6 to U3
Changed lines of the file:
@@
 $EndDescr
 $Comp
-L pspice:CAP C5
+L pspice:CAP C2
 U 1 1 61A64F42
 P 3600 3250
-F 0 "C5" H 3778 3296 50  0000 L CNN
+F 0 "C2" H 3778 3296 50  0000 L CNN
 F 1 "100u" H 3778 3205 50  0000 L CNN
 F 2 "Capacitor_SMD:CP_Elec_6.3x5.8" H 3600 3250 50  0001 C CNN
@@
 $EndComp
 $Comp
-L pspice:CAP C7
+L pspice:CAP C3
 U 1 1 61A6675D
 P 4700 3250
-F 0 "C7" H 4878 3296 50  0000 L CNN
+F 0 "C3" H 4878 3296 50  0000 L CNN
 F 1 "100u" H 4878 3205 50  0000 L CNN
 F 2 "Capacitor_SMD:CP_Elec_6.3x5.8" H 4700 3250 50  0001 C CNN
@@
 	4700 3500 4700 3850
 $Comp
-L Device:LED D7
+L Device:LED D3
 U 1 1 61A6F4A6
 P 5250 3600
-F 0 "D7" H 5243 3817 50  0000 C CNN
+F 0 "D3" H 5243 3817 50  0000 C CNN
 F 1 "LED" H 5243 3726 50  0000 C CNN
 F 2 "LED_SMD:LED_0805_2012Metric_Pad1.15x1.40mm_HandSolder" H 5250 3600 50  0001 C CNN
@@
 $EndComp
 $Comp
-L Device:R R14
+L Device:R R6
 U 1 1 61A71AC0
 P 5250 3250
-F 0 "R14" H 5320 3296 50  0000 L CNN
+F 0 "R6" H 5320 3296 50  0000 L CNN
 F 1 "680" H 5320 3205 50  0000 L CNN
 F 2 "Resistor_SMD:R_0805_2012Metric_Pad1.20x1.40mm_HandSolder" V 5180 3250 50  0001 C CNN
@@
 	5250 3450 5250 3400
 $Comp
-L Regulator_Linear:LM7805_TO220 U5
+L Regulator_Linear:LM7805_TO220 U2
 U 1 1 61A72BA8
 P 4200 2900
-F 0 "U5" H 4200 3142 50  0000 C CNN
+F 0 "U2" H 4200 3142 50  0000 C CNN
 F 1 "LM7805_TO220" H 4200 3051 50  0000 C CNN
 F 2 "Package_TO_SOT_THT:TO-220-3_Vertical" H 4200 3125 50  0001 C CIN
@@
 $EndComp
 $Comp
-L pspice:CAP C6
+L pspice:CAP C4
 U 1 1 61A8758A
 P 3600 4800
-F 0 "C6" H 3778 4846 50  0000 L CNN
+F 0 "C4" H 3778 4846 50  0000 L CNN
 F 1 "10u" H 3778 4755 50  0000 L CNN
 F 2 "Capacitor_SMD:C_1206_3216Metric_Pad1.33x1.80mm_HandSolder" H 3600 4800 50  0001 C CNN
@@
 $EndComp
 $Comp
-L pspice:CAP C8
+L pspice:CAP C5
 U 1 1 61A87590
 P 4700 4800
-F 0 "C8" H 4878 4846 50  0000 L CNN
+F 0 "C5" H 4878 4846 50  0000 L CNN
 F 1 "10u" H 4878 4755 50  0000 L CNN
 F 2 "Capacitor_SMD:C_1206_3216Metric_Pad1.33x1.80mm_HandSolder" H 4700 4800 50  0001 C CNN
@@
 	4700 5050 4700 5400
 $Comp
-L Device:LED D8
+L Device:LED D4
 U 1 1 61A875AB
 P 5250 5150
-F 0 "D8" H 5243 5367 50  0000 C CNN
+F 0 "D4" H 5243 5367 50  0000 C CNN
 F 1 "LED" H 5243 5276 50  0000 C CNN
 F 2 "LED_SMD:LED_0805_2012Metric_Pad1.15x1.40mm_HandSolder" H 5250 5150 50  0001 C CNN
@@
 $EndComp
 $Comp
-L Device:R R18
+L Device:R R7
 U 1 1 61A875B1
 P 5250 4800
-F 0 "R18" H 5320 4846 50  0000 L CNN
+F 0 "R7" H 5320 4846 50  0000 L CNN
 F 1 "470" H 5320 4755 50  0000 L CNN
 F 2 "Resistor_SMD:R_0805_2012Metric_Pad1.20x1.40mm_HandSolder" V 5180 4800 50  0001 C CNN
@@
 	5250 4450 5250 4650
 $Comp
-L Regulator_Linear:LM1117-3.3 U6
+L Regulator_Linear:LM1117-3.3 U3
 U 1 1 61A88682
 P 4200 4450
-F 0 "U6" H 4200 4692 50  0000 C CNN
+F 0 "U3" H 4200 4692 50  0000 C CNN
 F 1 "LM1117-3.3" H 4200 4601 50  0000 C CNN
 F 2 "Package_TO_SOT_THT:TO-220-3_Vertical" H 4200 4450 50  0001 C CNN
@@
 $EndComp
 $Comp
-L Device:R R13
+L Device:R R5
 U 1 1 61A8B0C5
 P 3350 2900
-F 0 "R13" H 3420 2946 50  0000 L CNN
+F 0 "R5" H 3420 2946 50  0000 L CNN
 F 1 "2" H 3420 2855 50  0000 L CNN
-F 2 "Resistor_SMD:R_0805_2012Metric_Pad1.20x1.40mm_HandSolder" V 3280 2900 50  0001 C CNN
+F 2 "Resistor_SMD:R_1210_3225Metric_Pad1.30x2.65mm_HandSolder" V 3280 2900 50  0001 C CNN
 F 3 "~" H 3350 2900 50  0001 C CNN
 	1    3350 2900
@@
 $EndComp
 $Comp
-L Transistor_BJT:TIP42C Q3
+L Transistor_BJT:TIP42C Q1
 U 1 1 61A8E37D
 P 3600 2500
-F 0 "Q3" H 3791 2546 50  0000 L CNN
+F 0 "Q1" H 3791 2546 50  0000 L CNN
 F 1 "TIP42C" H 3791 2455 50  0000 L CNN
 F 2 "Package_TO_SOT_THT:TO-220-3_Vertical" H 3850 2425 50  0001 L CIN
