File: Diseño PCB/PCB-ESP32S - reles/PCB-ESP32S.sch (KiCad schematic (older format))
At the start: 10 parts, among them J7 Screw_Terminal_01x03, SW1 SW_DIP_x01, SW2 SW_DIP_x01, U1 ESP-32S

Commit message: PCB2
Connections:
- net IO14: now reaches U1.13 (IO14)
- net IO12: now reaches U1.14 (IO12)
Changed lines of the file:
@@
 F3 "VCC_source" I L 9500 3700 50
 F4 "GND" I L 9500 3850 50
-F5 "IN1" I R 10250 3600 50
-F6 "IN2" I R 10250 3800 50
+F5 "GPIO1" I R 10250 3600 50
+F6 "GPIO2" I R 10250 3800 50
 $EndSheet
 Connection ~ 2800 2500
@@
 	4650 4850 4650 5200
 $Comp
-L power:+5V #PWR?
+L power:+5V #PWR0107
 U 1 1 61BFB68C
 P 3750 5600
-F 0 "#PWR?" H 3750 5450 50  0001 C CNN
+F 0 "#PWR0107" H 3750 5450 50  0001 C CNN
 F 1 "+5V" H 3765 5773 50  0000 C CNN
 F 2 "" H 3750 5600 50  0001 C CNN
@@
 $EndComp
 $Comp
-L power:+3.3V #PWR?
+L power:+3.3V #PWR0108
 U 1 1 61BFBED1
 P 3750 5800
-F 0 "#PWR?" H 3750 5650 50  0001 C CNN
+F 0 "#PWR0108" H 3750 5650 50  0001 C CNN
 F 1 "+3.3V" H 3765 5973 50  0000 C CNN
 F 2 "" H 3750 5800 50  0001 C CNN
@@
 	3750 5850 3750 5800
 $Comp
-L power:GND #PWR?
+L power:GND #PWR0109
 U 1 1 61C01E8D
 P 1900 6100
-F 0 "#PWR?" H 1900 5850 50  0001 C CNN
+F 0 "#PWR0109" H 1900 5850 50  0001 C CNN
 F 1 "GND" H 1905 5927 50  0000 C CNN
 F 2 "" H 1900 6100 50  0001 C CNN
@@
 $EndComp
 $Comp
-L power:GND #PWR?
+L power:GND #PWR0110
 U 1 1 61C02BAF
 P 9350 3950
-F 0 "#PWR?" H 9350 3700 50  0001 C CNN
+F 0 "#PWR0110" H 9350 3700 50  0001 C CNN
 F 1 "GND" H 9355 3777 50  0000 C CNN
 F 2 "" H 9350 3950 50  0001 C CNN
@@
 F5 "GND" I L 2100 6000 50
 $EndSheet
-Wire Wire Line
-	5550 4850 5650 4850
 $Comp
 L PCB-ESP32S-rescue:ESP-32S-ESP32S-PCB-ESP32S-rescue-PCB-ESP32S-rescue U1
@@
 	1    0    0    -1
 $EndComp
+$Comp
+L power:+5V #PWR0111
+U 1 1 61E10981
+P 9350 3550
+F 0 "#PWR0111" H 9350 3400 50  0001 C CNN
+F 1 "+5V" H 9365 3723 50  0000 C CNN
+F 2 "" H 9350 3550 50  0001 C CNN
+F 3 "" H 9350 3550 50  0001 C CNN
+	1    9350 3550
+	1    0    0    -1
+$EndComp
+Wire Wire Line
+	9500 3550 9350 3550
+Text GLabel 10350 3600 2    50   Input ~ 0
+IO12
+Text GLabel 10350 3800 2    50   Input ~ 0
+IO14
+Text GLabel 4050 4400 0    50   Input ~ 0
+IO12
+Text GLabel 4050 4300 0    50   Input ~ 0
+IO14
+Wire Wire Line
+	10250 3600 10350 3600
+Wire Wire Line
+	10250 3800 10350 3800
+Wire Wire Line
+	4150 4400 4050 4400
+Wire Wire Line
+	4150 4300 4050 4300
+$Comp
+L power:+12V #PWR0112
+U 1 1 61E183CC
+P 9200 3650
+F 0 "#PWR0112" H 9200 3500 50  0001 C CNN
+F 1 "+12V" H 9215 3823 50  0000 C CNN
+F 2 "" H 9200 3650 50  0001 C CNN
+F 3 "" H 9200 3650 50  0001 C CNN
+	1    9200 3650
+	1    0    0    -1
+$EndComp
+Wire Wire Line
+	9500 3700 9200 3700
+Wire Wire Line
+	9200 3700 9200 3650
+$Comp
+L power:+12V #PWR0113
+U 1 1 61E19E53
+P 1900 5300
+F 0 "#PWR0113" H 1900 5150 50  0001 C CNN
+F 1 "+12V" H 1915 5473 50  0000 C CNN
+F 2 "" H 1900 5300 50  0001 C CNN
+F 3 "" H 1900 5300 50  0001 C CNN
+	1    1900 5300
+	1    0    0    -1
+$EndComp
+Wire Wire Line
+	2100 5350 1900 5350
+Wire Wire Line
+	1900 5350 1900 5300
 $EndSCHEMATC

Commit message: PCB reles
Parts:
- added Cdes1: 100n, Capacitor_SMD:C_0805_2012Metric_Pad1.18x1.45mm_HandSolder, symbol charger_stepup-rescue:C
Connections:
- net +3V3: now also Cdes1.1
- net GND: now also Cdes1.2
Changed lines of the file:
@@
 Wire Wire Line
 	2800 3650 2800 3700
-Connection ~ 2800 2950
-Wire Wire Line
-	2800 3050 2800 2950
-Wire Wire Line
-	2800 2950 2800 2900
-Wire Wire Line
-	3250 2950 2800 2950
 Wire Wire Line
 	3250 3300 3250 2950
@@
 	2800 2500 2800 2600
 Wire Wire Line
-	3350 2500 2800 2500
+	3350 2500 3100 2500
 Wire Wire Line
 	3350 3200 3350 2500
@@
 	3800 3100 4150 3100
 Wire Wire Line
-	3800 2800 3800 3100
+	3800 2800 3800 2900
 $Comp
 L Device:R R1
@@
 	1    2800 2750
 	1    0    0    -1
-$EndComp
-$Comp
-L Switch:SW_DIP_x01 SW1
-U 1 1 619FF8A4
-P 2800 3350
-F 0 "SW1" H 2800 3617 50  0000 C CNN
-F 1 "SW_DIP_x01" H 2800 3526 50  0000 C CNN
-F 2 "Button_Switch_SMD:SW_SPST_SKQG_WithStem" H 2800 3350 50  0001 C CNN
-F 3 "~" H 2800 3350 50  0001 C CNN
-	1    2800 3350
-	0    -1   -1   0
 $EndComp
 $Comp
@@
 Wire Wire Line
 	1900 5350 1900 5300
+Connection ~ 3100 2500
+Wire Wire Line
+	3100 2500 2800 2500
+Wire Wire Line
+	3100 2600 3100 2500
+$Comp
+L Switch:SW_DIP_x01 SW1
+U 1 1 619FF8A4
+P 2800 3350
+F 0 "SW1" H 2800 3617 50  0000 C CNN
+F 1 "SW_DIP_x01" H 2800 3526 50  0000 C CNN
+F 2 "Button_Switch_SMD:SW_SPST_SKQG_WithStem" H 2800 3350 50  0001 C CNN
+F 3 "~" H 2800 3350 50  0001 C CNN
+	1    2800 3350
+	0    -1   -1   0
+$EndComp
+Connection ~ 2800 2950
+Wire Wire Line
+	2800 2950 2800 2900
+Wire Wire Line
+	2800 3050 2800 2950
+$Comp
+L charger_stepup-rescue:C Cdes1
+U 1 1 61E20FBD
+P 3100 2750
+F 0 "Cdes1" H 3215 2796 50  0000 L CNN
+F 1 "100n" H 3215 2705 50  0000 L CNN
+F 2 "Capacitor_SMD:C_0805_2012Metric_Pad1.18x1.45mm_HandSolder" H 3138 2600 50  0001 C CNN
+F 3 "" H 3100 2750 50  0001 C CNN
+	1    3100 2750
+	1    0    0    -1
+$EndComp
+Wire Wire Line
+	3250 2950 2800 2950
+Wire Wire Line
+	3100 2900 3800 2900
+Connection ~ 3800 2900
+Wire Wire Line
+	3800 2900 3800 3100
 $EndSCHEMATC

Commit message: PCBs ok
Parts:
- SW1, SW2: footprint Button_Switch_SMD:SW_SPST_SKQG_WithStem -> Button_Switch_SMD:SW_SPST_TL3305A
Changed lines of the file:
@@
 F 0 "SW2" H 7050 4717 50  0000 C CNN
 F 1 "SW_DIP_x01" H 7050 4626 50  0000 C CNN
-F 2 "Button_Switch_SMD:SW_SPST_SKQG_WithStem" H 7050 4450 50  0001 C CNN
+F 2 "Button_Switch_SMD:SW_SPST_TL3305A" H 7050 4450 50  0001 C CNN
 F 3 "~" H 7050 4450 50  0001 C CNN
 	1    7050 4450
@@
 F 0 "SW1" H 2800 3617 50  0000 C CNN
 F 1 "SW_DIP_x01" H 2800 3526 50  0000 C CNN
-F 2 "Button_Switch_SMD:SW_SPST_SKQG_WithStem" H 2800 3350 50  0001 C CNN
+F 2 "Button_Switch_SMD:SW_SPST_TL3305A" H 2800 3350 50  0001 C CNN
 F 3 "~" H 2800 3350 50  0001 C CNN
 	1    2800 3350

Commit message: PCB reles - GND plano
Changed lines of the file:
@@
 F1 "alimentacion.sch" 50
 F2 "5V" I R 3600 5650 50
-F3 "12V" I L 2100 5350 50
-F4 "3.3V" I R 3600 5850 50
-F5 "GND" I L 2100 6000 50
+F3 "3.3V" I R 3600 5850 50
+F4 "GND" I L 2100 6000 50
+F5 "+12V" I L 2100 5350 50
 $EndSheet
 $Comp

Commit message: dos pcb finalizadas
Parts:
- J1: renamed from J7; footprint TerminalBlock:TerminalBlock_bornier-3_P5.08mm -> Connector_JST:JST_GH_BM03B-GHS-TBT_1x03-1MP_P1.25mm_Vertical
- renumbered D9 to D1, D10 to D2, R16 to R2, R2 to R3, R17 to R4
Connections:
- net GND: now also U1.38 (GND)
Changed lines of the file:
@@
 $EndComp
 $Comp
-L Device:R R2
+L Device:R R3
 U 1 1 61A006CD
 P 6550 4150
-F 0 "R2" H 6620 4196 50  0000 L CNN
+F 0 "R3" H 6620 4196 50  0000 L CNN
 F 1 "12K" H 6620 4105 50  0000 L CNN
 F 2 "Resistor_SMD:R_0805_2012Metric_Pad1.20x1.40mm_HandSolder" V 6480 4150 50  0001 C CNN
@@
 $EndComp
 $Comp
-L Device:LED D10
+L Device:LED D2
 U 1 1 61BB5D8E
 P 6100 4650
-F 0 "D10" H 6093 4867 50  0000 C CNN
+F 0 "D2" H 6093 4867 50  0000 C CNN
 F 1 "LED" H 6093 4776 50  0000 C CNN
 F 2 "LED_SMD:LED_0805_2012Metric_Pad1.15x1.40mm_HandSolder" H 6100 4650 50  0001 C CNN
@@
 P 7250 3150
 AR Path="/61A61E97/61BBC590" Ref="J?"  Part="1"
-AR Path="/61BBC590" Ref="J7"  Part="1"
-F 0 "J7" H 7330 3192 50  0000 L CNN
+AR Path="/61BBC590" Ref="J1"  Part="1"
+F 0 "J1" H 7330 3192 50  0000 L CNN
 F 1 "Screw_Terminal_01x03" H 7330 3101 50  0000 L CNN
-F 2 "TerminalBlock:TerminalBlock_bornier-3_P5.08mm" H 7250 3150 50  0001 C CNN
+F 2 "Connector_JST:JST_GH_BM03B-GHS-TBT_1x03-1MP_P1.25mm_Vertical" H 7250 3150 50  0001 C CNN
 F 3 "~" H 7250 3150 50  0001 C CNN
 	1    7250 3150
@@
 $EndComp
 Wire Wire Line
-	6000 3050 6550 3050
+	6000 3050 6150 3050
 Wire Wire Line
 	6900 3550 6000 3550
@@
 	6550 3050 7050 3050
 $Comp
-L Device:R R17
+L Device:R R4
 U 1 1 61BC4B9D
 P 6350 4950
-F 0 "R17" H 6420 4996 50  0000 L CNN
+F 0 "R4" H 6420 4996 50  0000 L CNN
 F 1 "220" H 6420 4905 50  0000 L CNN
 F 2 "Resistor_SMD:R_0805_2012Metric_Pad1.20x1.40mm_HandSolder" V 6280 4950 50  0001 C CNN
@@
 	4750 4950 4750 4850
 $Comp
-L Device:LED D9
+L Device:LED D1
 U 1 1 61BC9643
 P 2250 2750
-F 0 "D9" H 2243 2967 50  0000 C CNN
+F 0 "D1" H 2243 2967 50  0000 C CNN
 F 1 "LED" H 2243 2876 50  0000 C CNN
 F 2 "LED_SMD:LED_0805_2012Metric_Pad1.15x1.40mm_HandSolder" H 2250 2750 50  0001 C CNN
@@
 $EndComp
 $Comp
-L Device:R R16
+L Device:R R2
 U 1 1 61BC9649
 P 2250 3100
-F 0 "R16" H 2320 3146 50  0000 L CNN
+F 0 "R2" H 2320 3146 50  0000 L CNN
 F 1 "220" H 2320 3055 50  0000 L CNN
 F 2 "Resistor_SMD:R_0805_2012Metric_Pad1.20x1.40mm_HandSolder" V 2180 3100 50  0001 C CNN
@@
 Wire Wire Line
 	3800 2900 3800 3100
+Wire Wire Line
+	6000 3150 6150 3150
+Wire Wire Line
+	6150 3150 6150 3050
+Connection ~ 6150 3050
+Wire Wire Line
+	6150 3050 6550 3050
 $EndSCHEMATC

Commit message: PCB relés, te lo juro por Dieguito Maradona :''v
Parts:
- J1: footprint Connector_JST:JST_GH_BM03B-GHS-TBT_1x03-1MP_P1.25mm_Vertical -> Connector_JST:JST_EH_B3B-EH-A_1x03_P2.50mm_Vertical
Changed lines of the file:
@@
 F 0 "J1" H 7330 3192 50  0000 L CNN
 F 1 "Screw_Terminal_01x03" H 7330 3101 50  0000 L CNN
-F 2 "Connector_JST:JST_GH_BM03B-GHS-TBT_1x03-1MP_P1.25mm_Vertical" H 7250 3150 50  0001 C CNN
+F 2 "Connector_JST:JST_EH_B3B-EH-A_1x03_P2.50mm_Vertical" H 7250 3150 50  0001 C CNN
 F 3 "~" H 7250 3150 50  0001 C CNN
 	1    7250 3150
